File: 8x8x8-RGB-LED-Cube-PCB/8x8x8-RGB-LED-Cube-PCB.kicad_pcb (KiCad board)
At the start: 2 copper layers, 290 x 290 mm, 0 parts

Commit message: PCB update
Parts:
- added C1: 0.1u, Capacitor_SMD:C_0603_1608Metric_Pad1.08x0.95mm_HandSolder, B.Cu at (180.5, 326.0)
- added C10: 0.1u, Capacitor_SMD:C_0603_1608Metric_Pad1.08x0.95mm_HandSolder, B.Cu at (67.0, 146.5)
- added C11: 0.1u, Capacitor_SMD:C_0603_1608Metric_Pad1.08x0.95mm_HandSolder, B.Cu at (67.0, 114.0)
- added C12: 0.1u, Capacitor_SMD:C_0603_1608Metric_Pad1.08x0.95mm_HandSolder, B.Cu at (67.0, 81.0)
- added C13: 0.1u, Capacitor_SMD:C_0603_1608Metric_Pad1.08x0.95mm_HandSolder, B.Cu at (82.0, 63.0)
- added C14: 0.1u, Capacitor_SMD:C_0603_1608Metric_Pad1.08x0.95mm_HandSolder, B.Cu at (115.0, 61.5)
- added C15: 0.1u, Capacitor_SMD:C_0603_1608Metric_Pad1.08x0.95mm_HandSolder, B.Cu at (148.0, 61.5)
- added C16: 0.1u, Capacitor_SMD:C_0603_1608Metric_Pad1.08x0.95mm_HandSolder, B.Cu at (175.6, 55.6)
- added C17: 0.1u, Capacitor_SMD:C_0603_1608Metric_Pad1.08x0.95mm_HandSolder, B.Cu at (212.5, 61.5)
- added C18: 0.1u, Capacitor_SMD:C_0603_1608Metric_Pad1.08x0.95mm_HandSolder, B.Cu at (241.1, 55.7)
- added C19: 0.1u, Capacitor_SMD:C_0603_1608Metric_Pad1.08x0.95mm_HandSolder, B.Cu at (279.0, 61.5)
- added C2: 0.1u, Capacitor_SMD:C_0603_1608Metric_Pad1.08x0.95mm_HandSolder, B.Cu at (147.5, 326.0)
- added C20: 0.1u, Capacitor_SMD:C_0603_1608Metric_Pad1.08x0.95mm_HandSolder, B.Cu at (312.0, 63.0)
- added C21: 0.1u, Capacitor_SMD:C_0603_1608Metric_Pad1.08x0.95mm_HandSolder, B.Cu at (327.0, 81.0)
- added C22: 0.1u, Capacitor_SMD:C_0603_1608Metric_Pad1.08x0.95mm_HandSolder, B.Cu at (327.0, 114.0)
- added C23: 0.1u, Capacitor_SMD:C_0603_1608Metric_Pad1.08x0.95mm_HandSolder, B.Cu at (327.0, 147.0)
- added C24: 0.1u, Capacitor_SMD:C_0603_1608Metric_Pad1.08x0.95mm_HandSolder, B.Cu at (327.0, 179.5)
- added C25: 0.1u, Capacitor_SMD:C_0603_1608Metric_Pad1.08x0.95mm_HandSolder, B.Cu at (327.0, 212.5)
- added C26: 0.1u, Capacitor_SMD:C_0603_1608Metric_Pad1.08x0.95mm_HandSolder, B.Cu at (327.0, 245.0)
- added C27: 0.1u, Capacitor_SMD:C_0603_1608Metric_Pad1.08x0.95mm_HandSolder, B.Cu at (327.0, 278.0)
- added C28: 0.1u, Capacitor_SMD:C_0603_1608Metric_Pad1.08x0.95mm_HandSolder, B.Cu at (328.0, 310.0)
- added C29: 0.1u, Capacitor_SMD:C_0603_1608Metric_Pad1.08x0.95mm_HandSolder, B.Cu at (312.0, 326.0)
- added C3: 0.1u, Capacitor_SMD:C_0603_1608Metric_Pad1.08x0.95mm_HandSolder, B.Cu at (115.0, 326.0)
- added C30: 0.1u, Capacitor_SMD:C_0603_1608Metric_Pad1.08x0.95mm_HandSolder, B.Cu at (279.0, 326.5)
- added C31: 0.1u, Capacitor_SMD:C_0603_1608Metric_Pad1.08x0.95mm_HandSolder, B.Cu at (246.0, 326.0)
- added C32: 0.1u, Capacitor_SMD:C_0603_1608Metric_Pad1.08x0.95mm_HandSolder, B.Cu at (213.5, 326.0)
- added C33: 0.1u, Capacitor_SMD:C_0603_1608Metric_Pad1.08x0.95mm_HandSolder, B.Cu at (8.75, 160.1)
- added C34: 0.1u, Capacitor_SMD:C_0603_1608Metric_Pad1.08x0.95mm_HandSolder, B.Cu at (121.5, 116.5)
- added C35: 0.1u, Capacitor_SMD:C_0603_1608Metric_Pad1.08x0.95mm_HandSolder, B.Cu at (181.5, 116.5)
- added C36: 0.1u, Capacitor_SMD:C_0603_1608Metric_Pad1.08x0.95mm_HandSolder, B.Cu at (241.5, 116.5)
- added C37: 0.1u, Capacitor_SMD:C_0603_1608Metric_Pad1.08x0.95mm_HandSolder, B.Cu at (152.5, 113.5)
- added C38: 0.1u, Capacitor_SMD:C_0603_1608Metric_Pad1.08x0.95mm_HandSolder, B.Cu at (212.5, 116.5)
- added C39: 0.1u, Capacitor_SMD:C_0603_1608Metric_Pad1.08x0.95mm_HandSolder, B.Cu at (272.5, 114.5)
- added C4: 0.1u, Capacitor_SMD:C_0603_1608Metric_Pad1.08x0.95mm_HandSolder, B.Cu at (82.0, 326.0)
- added C40: 0.1u, Capacitor_SMD:C_0603_1608Metric_Pad1.08x0.95mm_HandSolder, B.Cu at (121.5, 176.5)
- added C41: 0.1u, Capacitor_SMD:C_0603_1608Metric_Pad1.08x0.95mm_HandSolder, B.Cu at (-0.23, 170.6)
- added C42: 0.1u, Capacitor_SMD:C_0603_1608Metric_Pad1.08x0.95mm_HandSolder, B.Cu at (241.5, 176.5)
- added C43: 1000uF, Capacitor_SMD:CP_Elec_10x10.5, B.Cu at (184.6, 64.8)
- added C44: 0.1u, Capacitor_SMD:C_0603_1608Metric_Pad1.08x0.95mm_HandSolder, B.Cu at (152.5, 173.5)
- added C45: 0.1u, Capacitor_SMD:C_0603_1608Metric_Pad1.08x0.95mm_HandSolder, B.Cu at (212.5, 176.5)
- added C46: 0.1u, Capacitor_SMD:C_0603_1608Metric_Pad1.08x0.95mm_HandSolder, B.Cu at (272.5, 174.5)
- added C47: 0.1u, Capacitor_SMD:C_0603_1608Metric_Pad1.08x0.95mm_HandSolder, B.Cu at (121.5, 218.5)
- added C48: 0.1u, Capacitor_SMD:C_0603_1608Metric_Pad1.08x0.95mm_HandSolder, B.Cu at (181.5, 218.5)
- added C49: 0.1u, Capacitor_SMD:C_0603_1608Metric_Pad1.08x0.95mm_HandSolder, B.Cu at (241.5, 218.5)
- added C5: 0.1u, Capacitor_SMD:C_0603_1608Metric_Pad1.08x0.95mm_HandSolder, B.Cu at (67.0, 311.0)
- added C50: 0.1u, Capacitor_SMD:C_0603_1608Metric_Pad1.08x0.95mm_HandSolder, B.Cu at (152.5, 215.5)
- added C51: 0.1u, Capacitor_SMD:C_0603_1608Metric_Pad1.08x0.95mm_HandSolder, B.Cu at (212.5, 218.5)
- added C52: 0.1u, Capacitor_SMD:C_0603_1608Metric_Pad1.08x0.95mm_HandSolder, B.Cu at (272.5, 216.5)
- added C53: 0.1u, Capacitor_SMD:C_0603_1608Metric_Pad1.08x0.95mm_HandSolder, B.Cu at (121.5, 278.5)
- added C54: 0.1u, Capacitor_SMD:C_0603_1608Metric_Pad1.08x0.95mm_HandSolder, B.Cu at (181.5, 278.5)
- added C55: 0.1u, Capacitor_SMD:C_0603_1608Metric_Pad1.08x0.95mm_HandSolder, B.Cu at (241.5, 278.5)
- added C56: 0.1u, Capacitor_SMD:C_0603_1608Metric_Pad1.08x0.95mm_HandSolder, B.Cu at (152.5, 275.5)
- added C57: 0.1u, Capacitor_SMD:C_0603_1608Metric_Pad1.08x0.95mm_HandSolder, B.Cu at (212.5, 278.5)
- added C58: 0.1u, Capacitor_SMD:C_0603_1608Metric_Pad1.08x0.95mm_HandSolder, B.Cu at (272.5, 276.5)
- added C6: 0.1u, Capacitor_SMD:C_0603_1608Metric_Pad1.08x0.95mm_HandSolder, B.Cu at (67.0, 278.0)
- added C7: 0.1u, Capacitor_SMD:C_0603_1608Metric_Pad1.08x0.95mm_HandSolder, B.Cu at (67.0, 245.5)
- added C8: 0.1u, Capacitor_SMD:C_0603_1608Metric_Pad1.08x0.95mm_HandSolder, B.Cu at (67.0, 212.5)
- added C9: 0.1u, Capacitor_SMD:C_0603_1608Metric_Pad1.08x0.95mm_HandSolder, B.Cu at (67.0, 179.5)
- added D1: WS2812B, LED_SMD:LED_WS2812B_PLCC4_5.0x5.0mm_P3.2mm, B.Cu at (180.6, 331.0)
- added D10: WS2812B, LED_SMD:LED_WS2812B_PLCC4_5.0x5.0mm_P3.2mm, B.Cu at (62.0, 146.7)
- added D11: WS2812B, LED_SMD:LED_WS2812B_PLCC4_5.0x5.0mm_P3.2mm, B.Cu at (62.0, 113.9)
- added D12: WS2812B, LED_SMD:LED_WS2812B_PLCC4_5.0x5.0mm_P3.2mm, B.Cu at (62.0, 81.0)
- added D13: WS2812B, LED_SMD:LED_WS2812B_PLCC4_5.0x5.0mm_P3.2mm, B.Cu at (82.0, 58.0)
- added D14: WS2812B, LED_SMD:LED_WS2812B_PLCC4_5.0x5.0mm_P3.2mm, B.Cu at (114.9, 55.0)
- added D15: WS2812B, LED_SMD:LED_WS2812B_PLCC4_5.0x5.0mm_P3.2mm, B.Cu at (147.7, 55.0)
- added D16: WS2812B, LED_SMD:LED_WS2812B_PLCC4_5.0x5.0mm_P3.2mm, B.Cu at (180.6, 55.0)
- added D17: WS2812B, LED_SMD:LED_WS2812B_PLCC4_5.0x5.0mm_P3.2mm, B.Cu at (213.4, 55.0)
- added D18: WS2812B, LED_SMD:LED_WS2812B_PLCC4_5.0x5.0mm_P3.2mm, B.Cu at (246.3, 55.0)
- added D19: WS2812B, LED_SMD:LED_WS2812B_PLCC4_5.0x5.0mm_P3.2mm, B.Cu at (279.1, 55.0)
- added D2: WS2812B, LED_SMD:LED_WS2812B_PLCC4_5.0x5.0mm_P3.2mm, B.Cu at (147.7, 331.0)
- added D20: WS2812B, LED_SMD:LED_WS2812B_PLCC4_5.0x5.0mm_P3.2mm, B.Cu at (312.0, 58.0)
- added D21: WS2812B, LED_SMD:LED_WS2812B_PLCC4_5.0x5.0mm_P3.2mm, B.Cu at (332.0, 81.0)
- added D22: WS2812B, LED_SMD:LED_WS2812B_PLCC4_5.0x5.0mm_P3.2mm, B.Cu at (332.0, 113.9)
- added D23: WS2812B, LED_SMD:LED_WS2812B_PLCC4_5.0x5.0mm_P3.2mm, B.Cu at (332.0, 146.7)
- added D24: WS2812B, LED_SMD:LED_WS2812B_PLCC4_5.0x5.0mm_P3.2mm, B.Cu at (332.0, 179.6)
- added D25: WS2812B, LED_SMD:LED_WS2812B_PLCC4_5.0x5.0mm_P3.2mm, B.Cu at (332.0, 212.4)
- added D26: WS2812B, LED_SMD:LED_WS2812B_PLCC4_5.0x5.0mm_P3.2mm, B.Cu at (332.0, 245.3)
- added D27: WS2812B, LED_SMD:LED_WS2812B_PLCC4_5.0x5.0mm_P3.2mm, B.Cu at (332.0, 278.1)
- added D28: WS2812B, LED_SMD:LED_WS2812B_PLCC4_5.0x5.0mm_P3.2mm, B.Cu at (332.0, 311.0)
- added D29: WS2812B, LED_SMD:LED_WS2812B_PLCC4_5.0x5.0mm_P3.2mm, B.Cu at (312.0, 331.0)
- added D3: WS2812B, LED_SMD:LED_WS2812B_PLCC4_5.0x5.0mm_P3.2mm, B.Cu at (114.9, 331.0)
- added D30: WS2812B, LED_SMD:LED_WS2812B_PLCC4_5.0x5.0mm_P3.2mm, B.Cu at (279.1, 331.0)
- added D31: WS2812B, LED_SMD:LED_WS2812B_PLCC4_5.0x5.0mm_P3.2mm, B.Cu at (246.3, 331.0)
- added D32: WS2812B, LED_SMD:LED_WS2812B_PLCC4_5.0x5.0mm_P3.2mm, B.Cu at (213.4, 331.0)
- added D4: WS2812B, LED_SMD:LED_WS2812B_PLCC4_5.0x5.0mm_P3.2mm, B.Cu at (82.0, 331.0)
- added D5: WS2812B, LED_SMD:LED_WS2812B_PLCC4_5.0x5.0mm_P3.2mm, B.Cu at (62.0, 311.0)
- added D6: WS2812B, LED_SMD:LED_WS2812B_PLCC4_5.0x5.0mm_P3.2mm, B.Cu at (62.0, 278.1)
- added D7: WS2812B, LED_SMD:LED_WS2812B_PLCC4_5.0x5.0mm_P3.2mm, B.Cu at (62.0, 245.3)
- added D8: WS2812B, LED_SMD:LED_WS2812B_PLCC4_5.0x5.0mm_P3.2mm, B.Cu at (62.0, 212.4)
- added D9: WS2812B, LED_SMD:LED_WS2812B_PLCC4_5.0x5.0mm_P3.2mm, B.Cu at (62.0, 179.6)
- added DC1: Barrel_Jack_Switch, Connector_BarrelJack:BarrelJack_Horizontal, B.Cu at (197.0, 65.0)
- added ESP1: ESP32-DEVKITC-32D, ESP32-DEVKITC-32D:MODULE_ESP32-DEVKITC-32D, B.Cu at (244.0, 72.0)
- added H1: Wire_hole_1.2_2.5, LED-Cube:Wire_hole_1.5_2.8, F.Cu at (87.0, 100.0)
- added H10: Wire_hole_1.2_2.5, LED-Cube:Wire_hole_1.5_2.8, F.Cu at (122.0, 100.0)
- added H100: Wire_hole_1.2_2.5, LED-Cube:Wire_hole_1.5_2.8, F.Cu at (187.0, 202.0)
- added H101: Wire_hole_1.2_2.5, LED-Cube:Wire_hole_1.5_2.8, F.Cu at (217.0, 202.0)
- added H102: Wire_hole_1.2_2.5, LED-Cube:Wire_hole_1.5_2.8, F.Cu at (247.0, 202.0)
- added H103: Wire_hole_1.2_2.5, LED-Cube:Wire_hole_1.5_2.8, F.Cu at (277.0, 202.0)
- added H104: Wire_hole_1.2_2.5, LED-Cube:Wire_hole_1.5_2.8, F.Cu at (307.0, 202.0)
- added H105: Wire_hole_1.2_2.5, LED-Cube:Wire_hole_1.5_2.8, F.Cu at (92.0, 202.0)
- added H106: Wire_hole_1.2_2.5, LED-Cube:Wire_hole_1.5_2.8, F.Cu at (122.0, 202.0)
- added H107: Wire_hole_1.2_2.5, LED-Cube:Wire_hole_1.5_2.8, F.Cu at (152.0, 202.0)
- added H108: Wire_hole_1.2_2.5, LED-Cube:Wire_hole_1.5_2.8, F.Cu at (182.0, 202.0)
- added H109: Wire_hole_1.2_2.5, LED-Cube:Wire_hole_1.5_2.8, F.Cu at (212.0, 202.0)
- added H11: Wire_hole_1.2_2.5, LED-Cube:Wire_hole_1.5_2.8, F.Cu at (152.0, 100.0)
- added H110: Wire_hole_1.2_2.5, LED-Cube:Wire_hole_1.5_2.8, F.Cu at (242.0, 202.0)
- added H111: Wire_hole_1.2_2.5, LED-Cube:Wire_hole_1.5_2.8, F.Cu at (272.0, 202.0)
- added H112: Wire_hole_1.2_2.5, LED-Cube:Wire_hole_1.5_2.8, F.Cu at (302.0, 202.0)
- added H113: Wire_hole_1.2_2.5, LED-Cube:Wire_hole_1.5_2.8, F.Cu at (87.0, 202.0)
- added H114: Wire_hole_1.2_2.5, LED-Cube:Wire_hole_1.5_2.8, F.Cu at (117.0, 202.0)
- added H115: Wire_hole_1.2_2.5, LED-Cube:Wire_hole_1.5_2.8, F.Cu at (147.0, 202.0)
- added H116: Wire_hole_1.2_2.5, LED-Cube:Wire_hole_1.5_2.8, F.Cu at (177.0, 202.0)
- added H117: Wire_hole_1.2_2.5, LED-Cube:Wire_hole_1.5_2.8, F.Cu at (207.0, 202.0)
- added H118: Wire_hole_1.2_2.5, LED-Cube:Wire_hole_1.5_2.8, F.Cu at (237.0, 202.0)
- added H119: Wire_hole_1.2_2.5, LED-Cube:Wire_hole_1.5_2.8, F.Cu at (267.0, 202.0)
- added H12: Wire_hole_1.2_2.5, LED-Cube:Wire_hole_1.5_2.8, F.Cu at (182.0, 100.0)
- added H120: Wire_hole_1.2_2.5, LED-Cube:Wire_hole_1.5_2.8, F.Cu at (297.0, 202.0)
- added H121: Wire_hole_1.2_2.5, LED-Cube:Wire_hole_1.5_2.8, F.Cu at (97.0, 232.0)
- added H122: Wire_hole_1.2_2.5, LED-Cube:Wire_hole_1.5_2.8, F.Cu at (127.0, 232.0)
- added H123: Wire_hole_1.2_2.5, LED-Cube:Wire_hole_1.5_2.8, F.Cu at (157.0, 232.0)
- added H124: Wire_hole_1.2_2.5, LED-Cube:Wire_hole_1.5_2.8, F.Cu at (187.0, 232.0)
- added H125: Wire_hole_1.2_2.5, LED-Cube:Wire_hole_1.5_2.8, F.Cu at (217.0, 232.0)
- added H126: Wire_hole_1.2_2.5, LED-Cube:Wire_hole_1.5_2.8, F.Cu at (247.0, 232.0)
- added H127: Wire_hole_1.2_2.5, LED-Cube:Wire_hole_1.5_2.8, F.Cu at (277.0, 232.0)
- added H128: Wire_hole_1.2_2.5, LED-Cube:Wire_hole_1.5_2.8, F.Cu at (307.0, 232.0)
- added H129: Wire_hole_1.2_2.5, LED-Cube:Wire_hole_1.5_2.8, F.Cu at (92.0, 232.0)
- added H13: Wire_hole_1.2_2.5, LED-Cube:Wire_hole_1.5_2.8, F.Cu at (212.0, 100.0)
- added H130: Wire_hole_1.2_2.5, LED-Cube:Wire_hole_1.5_2.8, F.Cu at (122.0, 232.0)
- added H131: Wire_hole_1.2_2.5, LED-Cube:Wire_hole_1.5_2.8, F.Cu at (152.0, 232.0)
- added H132: Wire_hole_1.2_2.5, LED-Cube:Wire_hole_1.5_2.8, F.Cu at (182.0, 232.0)
- added H133: Wire_hole_1.2_2.5, LED-Cube:Wire_hole_1.5_2.8, F.Cu at (212.0, 232.0)
- added H134: Wire_hole_1.2_2.5, LED-Cube:Wire_hole_1.5_2.8, F.Cu at (242.0, 232.0)
- added H135: Wire_hole_1.2_2.5, LED-Cube:Wire_hole_1.5_2.8, F.Cu at (272.0, 232.0)
- added H136: Wire_hole_1.2_2.5, LED-Cube:Wire_hole_1.5_2.8, F.Cu at (302.0, 232.0)
- added H137: Wire_hole_1.2_2.5, LED-Cube:Wire_hole_1.5_2.8, F.Cu at (87.0, 232.0)
- added H138: Wire_hole_1.2_2.5, LED-Cube:Wire_hole_1.5_2.8, F.Cu at (117.0, 232.0)
- added H139: Wire_hole_1.2_2.5, LED-Cube:Wire_hole_1.5_2.8, F.Cu at (147.0, 232.0)
- added H14: Wire_hole_1.2_2.5, LED-Cube:Wire_hole_1.5_2.8, F.Cu at (242.0, 100.0)
- added H140: Wire_hole_1.2_2.5, LED-Cube:Wire_hole_1.5_2.8, F.Cu at (177.0, 232.0)
- added H141: Wire_hole_1.2_2.5, LED-Cube:Wire_hole_1.5_2.8, F.Cu at (207.0, 232.0)
- added H142: Wire_hole_1.2_2.5, LED-Cube:Wire_hole_1.5_2.8, F.Cu at (237.0, 232.0)
- added H143: Wire_hole_1.2_2.5, LED-Cube:Wire_hole_1.5_2.8, F.Cu at (267.0, 232.0)
- added H144: Wire_hole_1.2_2.5, LED-Cube:Wire_hole_1.5_2.8, F.Cu at (297.0, 232.0)
- added H145: Wire_hole_1.2_2.5, LED-Cube:Wire_hole_1.5_2.8, F.Cu at (97.0, 262.0)
- added H146: Wire_hole_1.2_2.5, LED-Cube:Wire_hole_1.5_2.8, F.Cu at (127.0, 262.0)
- added H147: Wire_hole_1.2_2.5, LED-Cube:Wire_hole_1.5_2.8, F.Cu at (157.0, 262.0)
- added H148: Wire_hole_1.2_2.5, LED-Cube:Wire_hole_1.5_2.8, F.Cu at (187.0, 262.0)
- added H149: Wire_hole_1.2_2.5, LED-Cube:Wire_hole_1.5_2.8, F.Cu at (217.0, 262.0)
- added H15: Wire_hole_1.2_2.5, LED-Cube:Wire_hole_1.5_2.8, F.Cu at (272.0, 100.0)
- added H150: Wire_hole_1.2_2.5, LED-Cube:Wire_hole_1.5_2.8, F.Cu at (247.0, 262.0)
- added H151: Wire_hole_1.2_2.5, LED-Cube:Wire_hole_1.5_2.8, F.Cu at (277.0, 262.0)
- added H152: Wire_hole_1.2_2.5, LED-Cube:Wire_hole_1.5_2.8, F.Cu at (307.0, 262.0)
- added H153: Wire_hole_1.2_2.5, LED-Cube:Wire_hole_1.5_2.8, F.Cu at (92.0, 262.0)
- added H154: Wire_hole_1.2_2.5, LED-Cube:Wire_hole_1.5_2.8, F.Cu at (122.0, 262.0)
- added H155: Wire_hole_1.2_2.5, LED-Cube:Wire_hole_1.5_2.8, F.Cu at (152.0, 262.0)
- added H156: Wire_hole_1.2_2.5, LED-Cube:Wire_hole_1.5_2.8, F.Cu at (182.0, 262.0)
- added H157: Wire_hole_1.2_2.5, LED-Cube:Wire_hole_1.5_2.8, F.Cu at (212.0, 262.0)
- added H158: Wire_hole_1.2_2.5, LED-Cube:Wire_hole_1.5_2.8, F.Cu at (242.0, 262.0)
- added H159: Wire_hole_1.2_2.5, LED-Cube:Wire_hole_1.5_2.8, F.Cu at (272.0, 262.0)
- added H16: Wire_hole_1.2_2.5, LED-Cube:Wire_hole_1.5_2.8, F.Cu at (302.0, 100.0)
- added H160: Wire_hole_1.2_2.5, LED-Cube:Wire_hole_1.5_2.8, F.Cu at (302.0, 262.0)
- added H161: Wire_hole_1.2_2.5, LED-Cube:Wire_hole_1.5_2.8, F.Cu at (87.0, 262.0)
- added H162: Wire_hole_1.2_2.5, LED-Cube:Wire_hole_1.5_2.8, F.Cu at (117.0, 262.0)
- added H163: Wire_hole_1.2_2.5, LED-Cube:Wire_hole_1.5_2.8, F.Cu at (147.0, 262.0)
- added H164: Wire_hole_1.2_2.5, LED-Cube:Wire_hole_1.5_2.8, F.Cu at (177.0, 262.0)
- added H165: Wire_hole_1.2_2.5, LED-Cube:Wire_hole_1.5_2.8, F.Cu at (207.0, 262.0)
- added H166: Wire_hole_1.2_2.5, LED-Cube:Wire_hole_1.5_2.8, F.Cu at (237.0, 262.0)
- added H167: Wire_hole_1.2_2.5, LED-Cube:Wire_hole_1.5_2.8, F.Cu at (267.0, 262.0)
- added H168: Wire_hole_1.2_2.5, LED-Cube:Wire_hole_1.5_2.8, F.Cu at (297.0, 262.0)
- added H169: Wire_hole_1.2_2.5, LED-Cube:Wire_hole_1.5_2.8, F.Cu at (97.0, 292.0)
- added H17: Wire_hole_1.2_2.5, LED-Cube:Wire_hole_1.5_2.8, F.Cu at (97.0, 100.0)
- added H170: Wire_hole_1.2_2.5, LED-Cube:Wire_hole_1.5_2.8, F.Cu at (127.0, 292.0)
- added H171: Wire_hole_1.2_2.5, LED-Cube:Wire_hole_1.5_2.8, F.Cu at (157.0, 292.0)
- added H172: Wire_hole_1.2_2.5, LED-Cube:Wire_hole_1.5_2.8, F.Cu at (187.0, 292.0)
- added H173: Wire_hole_1.2_2.5, LED-Cube:Wire_hole_1.5_2.8, F.Cu at (217.0, 292.0)
- added H174: Wire_hole_1.2_2.5, LED-Cube:Wire_hole_1.5_2.8, F.Cu at (247.0, 292.0)
- added H175: Wire_hole_1.2_2.5, LED-Cube:Wire_hole_1.5_2.8, F.Cu at (277.0, 292.0)
- added H176: Wire_hole_1.2_2.5, LED-Cube:Wire_hole_1.5_2.8, F.Cu at (307.0, 292.0)
- added H177: Wire_hole_1.2_2.5, LED-Cube:Wire_hole_1.5_2.8, F.Cu at (92.0, 292.0)
- added H178: Wire_hole_1.2_2.5, LED-Cube:Wire_hole_1.5_2.8, F.Cu at (122.0, 292.0)
- added H179: Wire_hole_1.2_2.5, LED-Cube:Wire_hole_1.5_2.8, F.Cu at (152.0, 292.0)
- added H18: Wire_hole_1.2_2.5, LED-Cube:Wire_hole_1.5_2.8, F.Cu at (127.0, 100.0)
- added H180: Wire_hole_1.2_2.5, LED-Cube:Wire_hole_1.5_2.8, F.Cu at (182.0, 292.0)
- added H181: Wire_hole_1.2_2.5, LED-Cube:Wire_hole_1.5_2.8, F.Cu at (212.0, 292.0)
- added H182: Wire_hole_1.2_2.5, LED-Cube:Wire_hole_1.5_2.8, F.Cu at (242.0, 292.0)
- added H183: Wire_hole_1.2_2.5, LED-Cube:Wire_hole_1.5_2.8, F.Cu at (272.0, 292.0)
- added H184: Wire_hole_1.2_2.5, LED-Cube:Wire_hole_1.5_2.8, F.Cu at (302.0, 292.0)
- added H185: Wire_hole_1.2_2.5, LED-Cube:Wire_hole_1.5_2.8, F.Cu at (87.0, 292.0)
- added H186: Wire_hole_1.2_2.5, LED-Cube:Wire_hole_1.5_2.8, F.Cu at (117.0, 292.0)
- added H187: Wire_hole_1.2_2.5, LED-Cube:Wire_hole_1.5_2.8, F.Cu at (147.0, 292.0)
- added H188: Wire_hole_1.2_2.5, LED-Cube:Wire_hole_1.5_2.8, F.Cu at (177.0, 292.0)
- added H189: Wire_hole_1.2_2.5, LED-Cube:Wire_hole_1.5_2.8, F.Cu at (207.0, 292.0)
- added H19: Wire_hole_1.2_2.5, LED-Cube:Wire_hole_1.5_2.8, F.Cu at (157.0, 100.0)
- added H190: Wire_hole_1.2_2.5, LED-Cube:Wire_hole_1.5_2.8, F.Cu at (237.0, 292.0)
- added H191: Wire_hole_1.2_2.5, LED-Cube:Wire_hole_1.5_2.8, F.Cu at (267.0, 292.0)
- added H192: Wire_hole_1.2_2.5, LED-Cube:Wire_hole_1.5_2.8, F.Cu at (297.0, 292.0)
- added H193: Wire_hole_1.2_2.5, LED-Cube:Wire_hole_1.5_2.8, F.Cu at (107.0, 89.0)
- added H194: Wire_hole_1.2_2.5, LED-Cube:Wire_hole_1.5_2.8, F.Cu at (137.0, 89.0)
- added H195: Wire_hole_1.2_2.5, LED-Cube:Wire_hole_1.5_2.8, F.Cu at (167.0, 89.0)
- added H196: Wire_hole_1.2_2.5, LED-Cube:Wire_hole_1.5_2.8, F.Cu at (194.0, 89.0)
- added H197: Wire_hole_1.2_2.5, LED-Cube:Wire_hole_1.5_2.8, F.Cu at (200.0, 89.0)
- added H198: Wire_hole_1.2_2.5, LED-Cube:Wire_hole_1.5_2.8, F.Cu at (227.0, 89.0)
- added H199: Wire_hole_1.2_2.5, LED-Cube:Wire_hole_1.5_2.8, F.Cu at (257.0, 89.0)
- added H2: Wire_hole_1.2_2.5, LED-Cube:Wire_hole_1.5_2.8, F.Cu at (117.0, 100.0)
- added H20: Wire_hole_1.2_2.5, LED-Cube:Wire_hole_1.5_2.8, F.Cu at (187.0, 100.0)
- added H200: Wire_hole_1.2_2.5, LED-Cube:Wire_hole_1.5_2.8, F.Cu at (287.0, 89.0)
- added H201: MountingHole, MountingHole:MountingHole_3.2mm_M3, F.Cu at (332.0, 331.0)
- added H202: MountingHole, MountingHole:MountingHole_3.2mm_M3, F.Cu at (62.0, 331.0)
- added H203: MountingHole, MountingHole:MountingHole_3.2mm_M3, F.Cu at (62.0, 61.0)
- added H204: MountingHole, MountingHole:MountingHole_3.2mm_M3, F.Cu at (332.0, 61.0)
- added H21: Wire_hole_1.2_2.5, LED-Cube:Wire_hole_1.5_2.8, F.Cu at (217.0, 100.0)
- added H22: Wire_hole_1.2_2.5, LED-Cube:Wire_hole_1.5_2.8, F.Cu at (247.0, 100.0)
- added H23: Wire_hole_1.2_2.5, LED-Cube:Wire_hole_1.5_2.8, F.Cu at (277.0, 100.0)
- added H24: Wire_hole_1.2_2.5, LED-Cube:Wire_hole_1.5_2.8, F.Cu at (307.0, 100.0)
- added H25: Wire_hole_1.2_2.5, LED-Cube:Wire_hole_1.5_2.8, F.Cu at (87.0, 130.0)
- added H26: Wire_hole_1.2_2.5, LED-Cube:Wire_hole_1.5_2.8, F.Cu at (117.0, 130.0)
- added H27: Wire_hole_1.2_2.5, LED-Cube:Wire_hole_1.5_2.8, F.Cu at (147.0, 130.0)
- added H28: Wire_hole_1.2_2.5, LED-Cube:Wire_hole_1.5_2.8, F.Cu at (177.0, 130.0)
- added H29: Wire_hole_1.2_2.5, LED-Cube:Wire_hole_1.5_2.8, F.Cu at (207.0, 130.0)
- added H3: Wire_hole_1.2_2.5, LED-Cube:Wire_hole_1.5_2.8, F.Cu at (147.0, 100.0)
- added H30: Wire_hole_1.2_2.5, LED-Cube:Wire_hole_1.5_2.8, F.Cu at (237.0, 130.0)
- added H31: Wire_hole_1.2_2.5, LED-Cube:Wire_hole_1.5_2.8, F.Cu at (267.0, 130.0)
- added H32: Wire_hole_1.2_2.5, LED-Cube:Wire_hole_1.5_2.8, F.Cu at (297.0, 130.0)
- added H33: Wire_hole_1.2_2.5, LED-Cube:Wire_hole_1.5_2.8, F.Cu at (92.0, 130.0)
- added H34: Wire_hole_1.2_2.5, LED-Cube:Wire_hole_1.5_2.8, F.Cu at (122.0, 130.0)
- added H35: Wire_hole_1.2_2.5, LED-Cube:Wire_hole_1.5_2.8, F.Cu at (152.0, 130.0)
- added H36: Wire_hole_1.2_2.5, LED-Cube:Wire_hole_1.5_2.8, F.Cu at (182.0, 130.0)
- added H37: Wire_hole_1.2_2.5, LED-Cube:Wire_hole_1.5_2.8, F.Cu at (212.0, 130.0)
- added H38: Wire_hole_1.2_2.5, LED-Cube:Wire_hole_1.5_2.8, F.Cu at (242.0, 130.0)
- added H39: Wire_hole_1.2_2.5, LED-Cube:Wire_hole_1.5_2.8, F.Cu at (272.0, 130.0)
- added H4: Wire_hole_1.2_2.5, LED-Cube:Wire_hole_1.5_2.8, F.Cu at (177.0, 100.0)
- added H40: Wire_hole_1.2_2.5, LED-Cube:Wire_hole_1.5_2.8, F.Cu at (302.0, 130.0)
- added H41: Wire_hole_1.2_2.5, LED-Cube:Wire_hole_1.5_2.8, F.Cu at (97.0, 130.0)
- added H42: Wire_hole_1.2_2.5, LED-Cube:Wire_hole_1.5_2.8, F.Cu at (127.0, 130.0)
- added H43: Wire_hole_1.2_2.5, LED-Cube:Wire_hole_1.5_2.8, F.Cu at (157.0, 130.0)
- added H44: Wire_hole_1.2_2.5, LED-Cube:Wire_hole_1.5_2.8, F.Cu at (187.0, 130.0)
- added H45: Wire_hole_1.2_2.5, LED-Cube:Wire_hole_1.5_2.8, F.Cu at (217.0, 130.0)
- added H46: Wire_hole_1.2_2.5, LED-Cube:Wire_hole_1.5_2.8, F.Cu at (247.0, 130.0)
- added H47: Wire_hole_1.2_2.5, LED-Cube:Wire_hole_1.5_2.8, F.Cu at (277.0, 130.0)
- added H48: Wire_hole_1.2_2.5, LED-Cube:Wire_hole_1.5_2.8, F.Cu at (307.0, 130.0)
- added H49: Wire_hole_1.2_2.5, LED-Cube:Wire_hole_1.5_2.8, F.Cu at (87.0, 160.0)
- added H5: Wire_hole_1.2_2.5, LED-Cube:Wire_hole_1.5_2.8, F.Cu at (207.0, 100.0)
- added H50: Wire_hole_1.2_2.5, LED-Cube:Wire_hole_1.5_2.8, F.Cu at (117.0, 160.0)
- added H51: Wire_hole_1.2_2.5, LED-Cube:Wire_hole_1.5_2.8, F.Cu at (147.0, 160.0)
- added H52: Wire_hole_1.2_2.5, LED-Cube:Wire_hole_1.5_2.8, F.Cu at (177.0, 160.0)
- added H53: Wire_hole_1.2_2.5, LED-Cube:Wire_hole_1.5_2.8, F.Cu at (207.0, 160.0)
- added H54: Wire_hole_1.2_2.5, LED-Cube:Wire_hole_1.5_2.8, F.Cu at (237.0, 160.0)
- added H55: Wire_hole_1.2_2.5, LED-Cube:Wire_hole_1.5_2.8, F.Cu at (267.0, 160.0)
- added H56: Wire_hole_1.2_2.5, LED-Cube:Wire_hole_1.5_2.8, F.Cu at (297.0, 160.0)
- added H57: Wire_hole_1.2_2.5, LED-Cube:Wire_hole_1.5_2.8, F.Cu at (92.0, 160.0)
- added H58: Wire_hole_1.2_2.5, LED-Cube:Wire_hole_1.5_2.8, F.Cu at (122.0, 160.0)
- added H59: Wire_hole_1.2_2.5, LED-Cube:Wire_hole_1.5_2.8, F.Cu at (152.0, 160.0)
- added H6: Wire_hole_1.2_2.5, LED-Cube:Wire_hole_1.5_2.8, F.Cu at (237.0, 100.0)
- added H60: Wire_hole_1.2_2.5, LED-Cube:Wire_hole_1.5_2.8, F.Cu at (182.0, 160.0)
- added H61: Wire_hole_1.2_2.5, LED-Cube:Wire_hole_1.5_2.8, F.Cu at (212.0, 160.0)
- added H62: Wire_hole_1.2_2.5, LED-Cube:Wire_hole_1.5_2.8, F.Cu at (242.0, 160.0)
- added H63: Wire_hole_1.2_2.5, LED-Cube:Wire_hole_1.5_2.8, F.Cu at (272.0, 160.0)
- added H64: Wire_hole_1.2_2.5, LED-Cube:Wire_hole_1.5_2.8, F.Cu at (302.0, 160.0)
- added H65: Wire_hole_1.2_2.5, LED-Cube:Wire_hole_1.5_2.8, F.Cu at (97.0, 160.0)
- added H66: Wire_hole_1.2_2.5, LED-Cube:Wire_hole_1.5_2.8, F.Cu at (127.0, 160.0)
- added H67: Wire_hole_1.2_2.5, LED-Cube:Wire_hole_1.5_2.8, F.Cu at (157.0, 160.0)
- added H68: Wire_hole_1.2_2.5, LED-Cube:Wire_hole_1.5_2.8, F.Cu at (187.0, 160.0)
- added H69: Wire_hole_1.2_2.5, LED-Cube:Wire_hole_1.5_2.8, F.Cu at (217.0, 160.0)
- added H7: Wire_hole_1.2_2.5, LED-Cube:Wire_hole_1.5_2.8, F.Cu at (267.0, 100.0)
- added H70: Wire_hole_1.2_2.5, LED-Cube:Wire_hole_1.5_2.8, F.Cu at (247.0, 160.0)
- added H71: Wire_hole_1.2_2.5, LED-Cube:Wire_hole_1.5_2.8, F.Cu at (277.0, 160.0)
- added H72: Wire_hole_1.2_2.5, LED-Cube:Wire_hole_1.5_2.8, F.Cu at (307.0, 160.0)
- added H73: Wire_hole_1.2_2.5, LED-Cube:Wire_hole_1.5_2.8, F.Cu at (87.0, 190.0)
- added H74: Wire_hole_1.2_2.5, LED-Cube:Wire_hole_1.5_2.8, F.Cu at (117.0, 190.0)
- added H75: Wire_hole_1.2_2.5, LED-Cube:Wire_hole_1.5_2.8, F.Cu at (147.0, 190.0)
- added H76: Wire_hole_1.2_2.5, LED-Cube:Wire_hole_1.5_2.8, F.Cu at (177.0, 190.0)
- added H77: Wire_hole_1.2_2.5, LED-Cube:Wire_hole_1.5_2.8, F.Cu at (207.0, 190.0)
- added H78: Wire_hole_1.2_2.5, LED-Cube:Wire_hole_1.5_2.8, F.Cu at (237.0, 190.0)
- added H79: Wire_hole_1.2_2.5, LED-Cube:Wire_hole_1.5_2.8, F.Cu at (267.0, 190.0)
- added H8: Wire_hole_1.2_2.5, LED-Cube:Wire_hole_1.5_2.8, F.Cu at (297.0, 100.0)
- added H80: Wire_hole_1.2_2.5, LED-Cube:Wire_hole_1.5_2.8, F.Cu at (297.0, 190.0)
- added H81: Wire_hole_1.2_2.5, LED-Cube:Wire_hole_1.5_2.8, F.Cu at (92.0, 190.0)
- added H82: Wire_hole_1.2_2.5, LED-Cube:Wire_hole_1.5_2.8, F.Cu at (122.0, 190.0)
- added H83: Wire_hole_1.2_2.5, LED-Cube:Wire_hole_1.5_2.8, F.Cu at (152.0, 190.0)
- added H84: Wire_hole_1.2_2.5, LED-Cube:Wire_hole_1.5_2.8, F.Cu at (182.0, 190.0)
- added H85: Wire_hole_1.2_2.5, LED-Cube:Wire_hole_1.5_2.8, F.Cu at (212.0, 190.0)
- added H86: Wire_hole_1.2_2.5, LED-Cube:Wire_hole_1.5_2.8, F.Cu at (242.0, 190.0)
- added H87: Wire_hole_1.2_2.5, LED-Cube:Wire_hole_1.5_2.8, F.Cu at (272.0, 190.0)
- added H88: Wire_hole_1.2_2.5, LED-Cube:Wire_hole_1.5_2.8, F.Cu at (302.0, 190.0)
- added H89: Wire_hole_1.2_2.5, LED-Cube:Wire_hole_1.5_2.8, F.Cu at (97.0, 190.0)
- added H9: Wire_hole_1.2_2.5, LED-Cube:Wire_hole_1.5_2.8, F.Cu at (92.0, 100.0)
- added H90: Wire_hole_1.2_2.5, LED-Cube:Wire_hole_1.5_2.8, F.Cu at (127.0, 190.0)
- added H91: Wire_hole_1.2_2.5, LED-Cube:Wire_hole_1.5_2.8, F.Cu at (157.0, 190.0)
- added H92: Wire_hole_1.2_2.5, LED-Cube:Wire_hole_1.5_2.8, F.Cu at (187.0, 190.0)
- added H93: Wire_hole_1.2_2.5, LED-Cube:Wire_hole_1.5_2.8, F.Cu at (217.0, 190.0)
- added H94: Wire_hole_1.2_2.5, LED-Cube:Wire_hole_1.5_2.8, F.Cu at (247.0, 190.0)
- added H95: Wire_hole_1.2_2.5, LED-Cube:Wire_hole_1.5_2.8, F.Cu at (277.0, 190.0)
- added H96: Wire_hole_1.2_2.5, LED-Cube:Wire_hole_1.5_2.8, F.Cu at (307.0, 190.0)
- added H97: Wire_hole_1.2_2.5, LED-Cube:Wire_hole_1.5_2.8, F.Cu at (97.0, 202.0)
- added H98: Wire_hole_1.2_2.5, LED-Cube:Wire_hole_1.5_2.8, F.Cu at (127.0, 202.0)
- added H99: Wire_hole_1.2_2.5, LED-Cube:Wire_hole_1.5_2.8, F.Cu at (157.0, 202.0)
- added PAD1: DATA, LED-Cube:Solder_pad_3x3mm, B.Cu at (214.0, 84.0)
- added PAD10: 2BOUT, LED-Cube:Solder_pad_3x3mm, B.Cu at (258.0, 111.0)
- added PAD11: 2RIN, LED-Cube:Solder_pad_3x3mm, B.Cu at (152.0, 110.0)
- added PAD12: 2GIN, LED-Cube:Solder_pad_3x3mm, B.Cu at (212.0, 112.5)
- added PAD13: 2BIN, LED-Cube:Solder_pad_3x3mm, B.Cu at (272.0, 111.0)
- added PAD14: 3ROUT, LED-Cube:Solder_pad_3x3mm, B.Cu at (136.0, 180.0)
- added PAD15: 3GOUT, LED-Cube:Solder_pad_3x3mm, B.Cu at (196.0, 180.0)
- added PAD16: 3BOUT, LED-Cube:Solder_pad_3x3mm, B.Cu at (256.0, 180.0)
- added PAD17: 3RIN, LED-Cube:Solder_pad_3x3mm, B.Cu at (122.0, 180.0)
- added PAD18: 3GIN, LED-Cube:Solder_pad_3x3mm, B.Cu at (182.0, 180.0)
- added PAD19: 3BIN, LED-Cube:Solder_pad_3x3mm, B.Cu at (242.0, 180.0)
- added PAD2: 1ROUT, LED-Cube:Solder_pad_3x3mm, B.Cu at (136.0, 120.0)
- added PAD20: 4ROUT, LED-Cube:Solder_pad_3x3mm, B.Cu at (138.0, 170.0)
- added PAD21: 4GOUT, LED-Cube:Solder_pad_3x3mm, B.Cu at (198.0, 172.5)
- added PAD22: 4BOUT, LED-Cube:Solder_pad_3x3mm, B.Cu at (258.0, 171.0)
- added PAD23: 4RIN, LED-Cube:Solder_pad_3x3mm, B.Cu at (152.0, 170.0)
- added PAD24: 4GIN, LED-Cube:Solder_pad_3x3mm, B.Cu at (212.0, 172.5)
- added PAD25: 4BIN, LED-Cube:Solder_pad_3x3mm, B.Cu at (272.0, 171.0)
- added PAD26: 5ROUT, LED-Cube:Solder_pad_3x3mm, B.Cu at (136.0, 222.0)
- added PAD27: 5GOUT, LED-Cube:Solder_pad_3x3mm, B.Cu at (196.0, 222.0)
- added PAD28: 5BOUT, LED-Cube:Solder_pad_3x3mm, B.Cu at (256.0, 222.0)
- added PAD29: 5RIN, LED-Cube:Solder_pad_3x3mm, B.Cu at (122.0, 222.0)
- added PAD3: 1GOUT, LED-Cube:Solder_pad_3x3mm, B.Cu at (196.0, 120.0)
- added PAD30: 5GIN, LED-Cube:Solder_pad_3x3mm, B.Cu at (182.0, 222.0)
- added PAD31: 5BIN, LED-Cube:Solder_pad_3x3mm, B.Cu at (242.0, 222.0)
- added PAD32: 6ROUT, LED-Cube:Solder_pad_3x3mm, B.Cu at (138.0, 212.0)
- added PAD33: 6GOUT, LED-Cube:Solder_pad_3x3mm, B.Cu at (198.0, 214.5)
- added PAD34: 6BOUT, LED-Cube:Solder_pad_3x3mm, B.Cu at (258.0, 213.0)
- added PAD35: 6RIN, LED-Cube:Solder_pad_3x3mm, B.Cu at (152.0, 212.0)
- added PAD36: 6GIN, LED-Cube:Solder_pad_3x3mm, B.Cu at (212.0, 214.5)
- added PAD37: 6BIN, LED-Cube:Solder_pad_3x3mm, B.Cu at (272.0, 213.0)
- added PAD38: 7ROUT, LED-Cube:Solder_pad_3x3mm, B.Cu at (136.0, 282.0)
- added PAD39: 7GOUT, LED-Cube:Solder_pad_3x3mm, B.Cu at (196.0, 282.0)
- added PAD4: 1BOUT, LED-Cube:Solder_pad_3x3mm, B.Cu at (256.0, 120.0)
- added PAD40: 7BOUT, LED-Cube:Solder_pad_3x3mm, B.Cu at (256.0, 282.0)
- added PAD41: 7RIN, LED-Cube:Solder_pad_3x3mm, B.Cu at (122.0, 282.0)
- added PAD42: 7GIN, LED-Cube:Solder_pad_3x3mm, B.Cu at (182.0, 282.0)
- added PAD43: 7BIN, LED-Cube:Solder_pad_3x3mm, B.Cu at (242.0, 282.0)
- added PAD44: 8ROUT, LED-Cube:Solder_pad_3x3mm, B.Cu at (138.0, 272.0)
- added PAD45: 8GOUT, LED-Cube:Solder_pad_3x3mm, B.Cu at (198.0, 274.5)
- added PAD46: 8BOUT, LED-Cube:Solder_pad_3x3mm, B.Cu at (258.0, 273.0)
- added PAD47: LAYEROUT, LED-Cube:Solder_pad_3x3mm, B.Cu at (-1.86, 219.5)
- added PAD48: 8RIN, LED-Cube:Solder_pad_3x3mm, B.Cu at (152.0, 272.0)
- added PAD49: 8GIN, LED-Cube:Solder_pad_3x3mm, B.Cu at (212.0, 274.5)
- added PAD5: 1RIN, LED-Cube:Solder_pad_3x3mm, B.Cu at (122.0, 120.0)
- added PAD50: 8BIN, LED-Cube:Solder_pad_3x3mm, B.Cu at (272.0, 273.0)
- added PAD51: LAYERIN, LED-Cube:Solder_pad_3x3mm, B.Cu at (-17.9, 227.5)
- added PAD52: Wire_pad, LED-Cube:Solder_pad_5x5mm, B.Cu at (208.0, 63.0)
- added PAD53: Wire_pad, LED-Cube:Solder_pad_5x5mm, B.Cu at (207.0, 56.0)
- added PAD6: 1GIN, LED-Cube:Solder_pad_3x3mm, B.Cu at (182.0, 120.0)
- added PAD7: 1BIN, LED-Cube:Solder_pad_3x3mm, B.Cu at (242.0, 120.0)
- added PAD8: 2ROUT, LED-Cube:Solder_pad_3x3mm, B.Cu at (138.0, 110.0)
- added PAD9: 2GOUT, LED-Cube:Solder_pad_3x3mm, B.Cu at (198.0, 112.5)
- added PAD98: Wire_pad, LED-Cube:Solder_pad_1.5x1.5mm, B.Cu at (328.5, 322.5)
- added PAD99: Wire_pad, LED-Cube:Solder_pad_1.5x1.5mm, B.Cu at (322.5, 325.5)
- added Q1: MMBT5551, Package_TO_SOT_SMD:SOT-23, B.Cu at (87.0, 92.0)
- added Q10: MMBT5551, Package_TO_SOT_SMD:SOT-23, B.Cu at (122.0, 92.0)
- added Q100: MMBT5551, Package_TO_SOT_SMD:SOT-23, B.Cu at (190.0, 198.0)
- added Q101: MMBT5551, Package_TO_SOT_SMD:SOT-23, B.Cu at (220.0, 198.0)
- added Q102: MMBT5551, Package_TO_SOT_SMD:SOT-23, B.Cu at (250.0, 198.0)
- added Q103: MMBT5551, Package_TO_SOT_SMD:SOT-23, B.Cu at (280.0, 198.0)
- added Q104: MMBT5551, Package_TO_SOT_SMD:SOT-23, B.Cu at (310.0, 198.0)
- added Q105: MMBT5551, Package_TO_SOT_SMD:SOT-23, B.Cu at (93.5, 198.0)
- added Q106: MMBT5551, Package_TO_SOT_SMD:SOT-23, B.Cu at (123.5, 198.0)
- added Q107: MMBT5551, Package_TO_SOT_SMD:SOT-23, B.Cu at (153.5, 198.0)
- added Q108: MMBT5551, Package_TO_SOT_SMD:SOT-23, B.Cu at (183.5, 198.0)
- added Q109: MMBT5551, Package_TO_SOT_SMD:SOT-23, B.Cu at (213.5, 198.0)
- added Q11: MMBT5551, Package_TO_SOT_SMD:SOT-23, B.Cu at (152.0, 92.0)
- added Q110: MMBT5551, Package_TO_SOT_SMD:SOT-23, B.Cu at (243.5, 198.0)
- added Q111: MMBT5551, Package_TO_SOT_SMD:SOT-23, B.Cu at (273.5, 198.0)
- added Q112: MMBT5551, Package_TO_SOT_SMD:SOT-23, B.Cu at (303.5, 198.0)
- added Q113: MMBT5551, Package_TO_SOT_SMD:SOT-23, B.Cu at (87.0, 198.0)
- added Q114: MMBT5551, Package_TO_SOT_SMD:SOT-23, B.Cu at (117.0, 198.0)
- added Q115: MMBT5551, Package_TO_SOT_SMD:SOT-23, B.Cu at (147.0, 198.0)
- added Q116: MMBT5551, Package_TO_SOT_SMD:SOT-23, B.Cu at (177.0, 198.0)
- added Q117: MMBT5551, Package_TO_SOT_SMD:SOT-23, B.Cu at (207.0, 198.0)
- added Q118: MMBT5551, Package_TO_SOT_SMD:SOT-23, B.Cu at (237.0, 198.0)
- added Q119: MMBT5551, Package_TO_SOT_SMD:SOT-23, B.Cu at (267.0, 198.0)
- added Q12: MMBT5551, Package_TO_SOT_SMD:SOT-23, B.Cu at (182.0, 92.0)
- added Q120: MMBT5551, Package_TO_SOT_SMD:SOT-23, B.Cu at (297.0, 198.0)
- added Q121: MMBT5551, Package_TO_SOT_SMD:SOT-23, B.Cu at (97.0, 240.0)
- added Q122: MMBT5551, Package_TO_SOT_SMD:SOT-23, B.Cu at (127.0, 240.0)
- added Q123: MMBT5551, Package_TO_SOT_SMD:SOT-23, B.Cu at (157.0, 240.0)
- added Q124: MMBT5551, Package_TO_SOT_SMD:SOT-23, B.Cu at (187.0, 240.0)
- added Q125: MMBT5551, Package_TO_SOT_SMD:SOT-23, B.Cu at (217.0, 240.0)
- added Q126: MMBT5551, Package_TO_SOT_SMD:SOT-23, B.Cu at (247.0, 240.0)
- added Q127: MMBT5551, Package_TO_SOT_SMD:SOT-23, B.Cu at (277.0, 240.0)
- added Q128: MMBT5551, Package_TO_SOT_SMD:SOT-23, B.Cu at (307.0, 240.0)
- added Q129: MMBT5551, Package_TO_SOT_SMD:SOT-23, B.Cu at (92.0, 240.0)
- added Q13: MMBT5551, Package_TO_SOT_SMD:SOT-23, B.Cu at (212.0, 92.0)
- added Q130: MMBT5551, Package_TO_SOT_SMD:SOT-23, B.Cu at (122.0, 240.0)
- added Q131: MMBT5551, Package_TO_SOT_SMD:SOT-23, B.Cu at (152.0, 240.0)
- added Q132: MMBT5551, Package_TO_SOT_SMD:SOT-23, B.Cu at (182.0, 240.0)
- added Q133: MMBT5551, Package_TO_SOT_SMD:SOT-23, B.Cu at (212.0, 240.0)
- added Q134: MMBT5551, Package_TO_SOT_SMD:SOT-23, B.Cu at (242.0, 240.0)
- added Q135: MMBT5551, Package_TO_SOT_SMD:SOT-23, B.Cu at (272.0, 240.0)
- added Q136: MMBT5551, Package_TO_SOT_SMD:SOT-23, B.Cu at (302.0, 240.0)
- added Q137: MMBT5551, Package_TO_SOT_SMD:SOT-23, B.Cu at (87.0, 240.0)
- added Q138: MMBT5551, Package_TO_SOT_SMD:SOT-23, B.Cu at (117.0, 240.0)
- added Q139: MMBT5551, Package_TO_SOT_SMD:SOT-23, B.Cu at (147.0, 240.0)
- added Q14: MMBT5551, Package_TO_SOT_SMD:SOT-23, B.Cu at (242.0, 92.0)
- added Q140: MMBT5551, Package_TO_SOT_SMD:SOT-23, B.Cu at (177.0, 240.0)
- added Q141: MMBT5551, Package_TO_SOT_SMD:SOT-23, B.Cu at (207.0, 240.0)
- added Q142: MMBT5551, Package_TO_SOT_SMD:SOT-23, B.Cu at (237.0, 240.0)
- added Q143: MMBT5551, Package_TO_SOT_SMD:SOT-23, B.Cu at (267.0, 240.0)
- added Q144: MMBT5551, Package_TO_SOT_SMD:SOT-23, B.Cu at (297.0, 240.0)
- added Q145: MMBT5551, Package_TO_SOT_SMD:SOT-23, B.Cu at (97.0, 254.0)
- added Q146: MMBT5551, Package_TO_SOT_SMD:SOT-23, B.Cu at (127.0, 254.0)
- added Q147: MMBT5551, Package_TO_SOT_SMD:SOT-23, B.Cu at (157.0, 254.0)
- added Q148: MMBT5551, Package_TO_SOT_SMD:SOT-23, B.Cu at (187.0, 254.0)
- added Q149: MMBT5551, Package_TO_SOT_SMD:SOT-23, B.Cu at (217.0, 254.0)
- added Q15: MMBT5551, Package_TO_SOT_SMD:SOT-23, B.Cu at (272.0, 92.0)
- added Q150: MMBT5551, Package_TO_SOT_SMD:SOT-23, B.Cu at (247.0, 254.0)
- added Q151: MMBT5551, Package_TO_SOT_SMD:SOT-23, B.Cu at (277.0, 254.0)
- added Q152: MMBT5551, Package_TO_SOT_SMD:SOT-23, B.Cu at (307.0, 254.0)
- added Q153: MMBT5551, Package_TO_SOT_SMD:SOT-23, B.Cu at (92.0, 254.0)
- added Q154: MMBT5551, Package_TO_SOT_SMD:SOT-23, B.Cu at (122.0, 254.0)
- added Q155: MMBT5551, Package_TO_SOT_SMD:SOT-23, B.Cu at (152.0, 254.0)
- added Q156: MMBT5551, Package_TO_SOT_SMD:SOT-23, B.Cu at (182.0, 254.0)
- added Q157: MMBT5551, Package_TO_SOT_SMD:SOT-23, B.Cu at (212.0, 254.0)
- added Q158: MMBT5551, Package_TO_SOT_SMD:SOT-23, B.Cu at (242.0, 254.0)
- added Q159: MMBT5551, Package_TO_SOT_SMD:SOT-23, B.Cu at (272.0, 254.0)
- added Q16: MMBT5551, Package_TO_SOT_SMD:SOT-23, B.Cu at (302.0, 92.0)
- added Q160: MMBT5551, Package_TO_SOT_SMD:SOT-23, B.Cu at (302.0, 254.0)
- added Q161: MMBT5551, Package_TO_SOT_SMD:SOT-23, B.Cu at (87.0, 254.0)
- added Q162: MMBT5551, Package_TO_SOT_SMD:SOT-23, B.Cu at (117.0, 254.0)
- added Q163: MMBT5551, Package_TO_SOT_SMD:SOT-23, B.Cu at (147.0, 254.0)
- added Q164: MMBT5551, Package_TO_SOT_SMD:SOT-23, B.Cu at (177.0, 254.0)
- added Q165: MMBT5551, Package_TO_SOT_SMD:SOT-23, B.Cu at (207.0, 254.0)
- added Q166: MMBT5551, Package_TO_SOT_SMD:SOT-23, B.Cu at (237.0, 254.0)
- added Q167: MMBT5551, Package_TO_SOT_SMD:SOT-23, B.Cu at (267.0, 254.0)
- added Q168: MMBT5551, Package_TO_SOT_SMD:SOT-23, B.Cu at (297.0, 254.0)
- added Q169: MMBT5551, Package_TO_SOT_SMD:SOT-23, B.Cu at (97.0, 300.0)
- added Q17: MMBT5551, Package_TO_SOT_SMD:SOT-23, B.Cu at (97.0, 92.0)
- added Q170: MMBT5551, Package_TO_SOT_SMD:SOT-23, B.Cu at (127.0, 300.0)
- added Q171: MMBT5551, Package_TO_SOT_SMD:SOT-23, B.Cu at (157.0, 300.0)
- added Q172: MMBT5551, Package_TO_SOT_SMD:SOT-23, B.Cu at (187.0, 300.0)
- added Q173: MMBT5551, Package_TO_SOT_SMD:SOT-23, B.Cu at (217.0, 300.0)
- added Q174: MMBT5551, Package_TO_SOT_SMD:SOT-23, B.Cu at (247.0, 300.0)
- added Q175: MMBT5551, Package_TO_SOT_SMD:SOT-23, B.Cu at (277.0, 300.0)
- added Q176: MMBT5551, Package_TO_SOT_SMD:SOT-23, B.Cu at (307.0, 300.0)
- added Q177: MMBT5551, Package_TO_SOT_SMD:SOT-23, B.Cu at (92.0, 300.0)
- added Q178: MMBT5551, Package_TO_SOT_SMD:SOT-23, B.Cu at (122.0, 300.0)
- added Q179: MMBT5551, Package_TO_SOT_SMD:SOT-23, B.Cu at (152.0, 300.0)
- added Q18: MMBT5551, Package_TO_SOT_SMD:SOT-23, B.Cu at (127.0, 92.0)
- added Q180: MMBT5551, Package_TO_SOT_SMD:SOT-23, B.Cu at (182.0, 300.0)
- added Q181: MMBT5551, Package_TO_SOT_SMD:SOT-23, B.Cu at (212.0, 300.0)
- added Q182: MMBT5551, Package_TO_SOT_SMD:SOT-23, B.Cu at (242.0, 300.0)
- added Q183: MMBT5551, Package_TO_SOT_SMD:SOT-23, B.Cu at (272.0, 300.0)
- added Q184: MMBT5551, Package_TO_SOT_SMD:SOT-23, B.Cu at (302.0, 300.0)
- added Q185: MMBT5551, Package_TO_SOT_SMD:SOT-23, B.Cu at (87.0, 300.0)
- added Q186: MMBT5551, Package_TO_SOT_SMD:SOT-23, B.Cu at (117.0, 300.0)
- added Q187: MMBT5551, Package_TO_SOT_SMD:SOT-23, B.Cu at (147.0, 300.0)
- added Q188: MMBT5551, Package_TO_SOT_SMD:SOT-23, B.Cu at (177.0, 300.0)
- added Q189: MMBT5551, Package_TO_SOT_SMD:SOT-23, B.Cu at (207.0, 300.0)
- added Q19: MMBT5551, Package_TO_SOT_SMD:SOT-23, B.Cu at (157.0, 92.0)
- added Q190: MMBT5551, Package_TO_SOT_SMD:SOT-23, B.Cu at (237.0, 300.0)
- added Q191: MMBT5551, Package_TO_SOT_SMD:SOT-23, B.Cu at (267.0, 300.0)
- added Q192: MMBT5551, Package_TO_SOT_SMD:SOT-23, B.Cu at (297.0, 300.0)
- added Q193: IRLML6401, Package_TO_SOT_SMD:SOT-23, B.Cu at (107.0, 92.5)
- added Q194: IRLML6401, Package_TO_SOT_SMD:SOT-23, B.Cu at (137.0, 92.5)
- added Q195: IRLML6401, Package_TO_SOT_SMD:SOT-23, B.Cu at (167.0, 92.5)
- added Q196: IRLML6401, Package_TO_SOT_SMD:SOT-23, B.Cu at (194.0, 92.5)
- added Q197: MMBT5551, Package_TO_SOT_SMD:SOT-23, B.Cu at (107.0, 98.0)
- added Q198: MMBT5551, Package_TO_SOT_SMD:SOT-23, B.Cu at (137.0, 98.0)
- added Q199: MMBT5551, Package_TO_SOT_SMD:SOT-23, B.Cu at (167.0, 98.0)
- added Q2: MMBT5551, Package_TO_SOT_SMD:SOT-23, B.Cu at (117.0, 92.0)
- added Q20: MMBT5551, Package_TO_SOT_SMD:SOT-23, B.Cu at (187.0, 92.0)
- added Q200: MMBT5551, Package_TO_SOT_SMD:SOT-23, B.Cu at (194.0, 98.0)
- added Q201: IRLML6401, Package_TO_SOT_SMD:SOT-23, B.Cu at (200.0, 92.5)
- added Q202: IRLML6401, Package_TO_SOT_SMD:SOT-23, B.Cu at (227.0, 92.5)
- added Q203: IRLML6401, Package_TO_SOT_SMD:SOT-23, B.Cu at (257.0, 92.5)
- added Q204: IRLML6401, Package_TO_SOT_SMD:SOT-23, B.Cu at (287.0, 92.5)
- added Q205: MMBT5551, Package_TO_SOT_SMD:SOT-23, B.Cu at (200.0, 98.0)
- added Q206: MMBT5551, Package_TO_SOT_SMD:SOT-23, B.Cu at (227.0, 98.0)
- added Q207: MMBT5551, Package_TO_SOT_SMD:SOT-23, B.Cu at (257.0, 98.0)
- added Q208: MMBT5551, Package_TO_SOT_SMD:SOT-23, B.Cu at (287.0, 98.0)
- added Q21: MMBT5551, Package_TO_SOT_SMD:SOT-23, B.Cu at (217.0, 92.0)
- added Q22: MMBT5551, Package_TO_SOT_SMD:SOT-23, B.Cu at (247.0, 92.0)
- added Q23: MMBT5551, Package_TO_SOT_SMD:SOT-23, B.Cu at (277.0, 92.0)
- added Q24: MMBT5551, Package_TO_SOT_SMD:SOT-23, B.Cu at (307.0, 92.0)
- added Q25: MMBT5551, Package_TO_SOT_SMD:SOT-23, B.Cu at (87.0, 138.0)
- added Q26: MMBT5551, Package_TO_SOT_SMD:SOT-23, B.Cu at (117.0, 138.0)
- added Q27: MMBT5551, Package_TO_SOT_SMD:SOT-23, B.Cu at (147.0, 138.0)
- added Q28: MMBT5551, Package_TO_SOT_SMD:SOT-23, B.Cu at (177.0, 138.0)
- added Q29: MMBT5551, Package_TO_SOT_SMD:SOT-23, B.Cu at (207.0, 138.0)
- added Q3: MMBT5551, Package_TO_SOT_SMD:SOT-23, B.Cu at (147.0, 92.0)
- added Q30: MMBT5551, Package_TO_SOT_SMD:SOT-23, B.Cu at (237.0, 138.0)
- added Q31: MMBT5551, Package_TO_SOT_SMD:SOT-23, B.Cu at (267.0, 138.0)
- added Q32: MMBT5551, Package_TO_SOT_SMD:SOT-23, B.Cu at (297.0, 138.0)
- added Q33: MMBT5551, Package_TO_SOT_SMD:SOT-23, B.Cu at (92.0, 138.0)
- added Q34: MMBT5551, Package_TO_SOT_SMD:SOT-23, B.Cu at (122.0, 138.0)
- added Q35: MMBT5551, Package_TO_SOT_SMD:SOT-23, B.Cu at (152.0, 138.0)
- added Q36: MMBT5551, Package_TO_SOT_SMD:SOT-23, B.Cu at (182.0, 138.0)
- added Q37: MMBT5551, Package_TO_SOT_SMD:SOT-23, B.Cu at (212.0, 138.0)
- added Q38: MMBT5551, Package_TO_SOT_SMD:SOT-23, B.Cu at (242.0, 138.0)
- added Q39: MMBT5551, Package_TO_SOT_SMD:SOT-23, B.Cu at (272.0, 138.0)
- added Q4: MMBT5551, Package_TO_SOT_SMD:SOT-23, B.Cu at (177.0, 92.0)
- added Q40: MMBT5551, Package_TO_SOT_SMD:SOT-23, B.Cu at (302.0, 138.0)
- added Q41: MMBT5551, Package_TO_SOT_SMD:SOT-23, B.Cu at (97.0, 138.0)
- added Q42: MMBT5551, Package_TO_SOT_SMD:SOT-23, B.Cu at (127.0, 138.0)
- added Q43: MMBT5551, Package_TO_SOT_SMD:SOT-23, B.Cu at (157.0, 138.0)
- added Q44: MMBT5551, Package_TO_SOT_SMD:SOT-23, B.Cu at (187.0, 138.0)
- added Q45: MMBT5551, Package_TO_SOT_SMD:SOT-23, B.Cu at (217.0, 138.0)
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Routing:
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- added copper zone on B.Cu, net GND
- added copper zone on F.Cu, net GND
Other:
- net class Default: trace_width 0.25 -> 0.254; via_dia 0.8 -> 0.45; via_drill 0.4 -> 0.25
- rule trace_min: 0.15 -> 0.254
- rule via_min_drill: 0.3 -> 0.2
