File: 8x8x8-RGB-LED-Cube-PCB/8x8x8-RGB-LED-Cube-PCB.sch (KiCad schematic (older format))
At the start: 422 parts, among them Q1 MMBT5551, SW1 SW_MEC_5E, SW2 SW_MEC_5E, SW3 SW_MEC_5E, SW4 SW_MEC_5E, SW5 SW_MEC_5E, U1 74HC595, U10 74HC595, U11 74HC595, U12 74HC595, U13 74HC595, U14 74HC595, U15 74HC595, U16 74HC595, U17 74HC595, U18 74HC595, U19 74HC595, U2 74HC595, U20 74HC595, U21 74HC595, U22 74HC595, U23 74HC595, U24 74HC595, U25 74HC595, U3 74HC595, U4 74HC595, U5 74HC595, U6 74HC595, U7 74HC595, U8 74HC595, U9 74HC595

Commit message: PCB update
Parts:
- added C1, C10, C12, C13, C14, C15, C16, C17, C18, C19, C2, C20, C21, C22, C23, C24, C25, C26, C3, C4, C5, C6, C7, C8, C9: 0.1u, Capacitor_SMD:C_0603_1608Metric_Pad1.08x0.95mm_HandSolder, symbol Device:C
- added C? (x32): 0.1u, symbol Device:C
- added D? (x32): WS2812B, LED_SMD:LED_WS2812B_PLCC4_5.0x5.0mm_P3.2mm, symbol LED:WS2812B
- added Q113, Q114, Q115, Q116, Q117, Q118, Q119, Q120, Q137, Q138, Q139, Q140, Q141, Q142, Q143, Q144, Q161, Q162, Q163, Q164, Q165, Q166, Q167, Q168, Q17, Q18, Q185, Q186, Q187, Q188, Q189, Q19, Q190, Q191, Q192, Q20, Q21, Q22, Q23, Q24, Q41, Q42, Q43, Q44, Q45, Q46, Q47, Q48, Q65, Q66, Q67, Q68, Q69, Q70, Q71, Q72, Q89, Q90, Q91, Q92, Q93, Q94, Q95, Q96, Q? (x8): MMBT5551, Package_TO_SOT_SMD:SOT-23_Handsoldering, symbol Device:Q_NPN_BEC
- added Q? (x8): IRLML6401, Package_TO_SOT_SMD:SOT-23, symbol Transistor_FET:IRLML6402
- added R113, R114, R115, R116, R117, R118, R119, R120, R161, R162, R163, R164, R165, R166, R167, R168, R17, R18, R19, R20, R209, R21, R210, R211, R212, R213, R214, R215, R216, R22, R23, R24, R257, R258, R259, R260, R261, R262, R263, R264, R305, R306, R307, R308, R309, R310, R311, R312, R353, R354, R355, R356, R357, R358, R359, R360, R65, R66, R67, R68, R69, R70, R71, R72: 665, Resistor_SMD:R_0805_2012Metric_Pad1.20x1.40mm_HandSolder, symbol Device:R_Small_US
- added R137, R138, R139, R140, R141, R142, R143, R144, R185, R186, R187, R188, R189, R190, R191, R192, R233, R234, R235, R236, R237, R238, R239, R240, R281, R282, R283, R284, R285, R286, R287, R288, R329, R330, R331, R332, R333, R334, R335, R336, R377, R378, R379, R380, R381, R382, R383, R384, R41, R42, R43, R44, R45, R46, R47, R48, R89, R90, R91, R92, R93, R94, R95, R96: 10k, Resistor_SMD:R_0603_1608Metric_Pad0.98x0.95mm_HandSolder, symbol Device:R_Small_US
- added R385, R386, R387, R388, R389: 10k, Resistor_SMD:R_0603_1608Metric_Pad0.98x0.95mm_HandSolder, symbol Device:R_US
- added R? (x16): 10k, symbol Device:R_US
- added R? (x8): 100, symbol Device:R_US
- C11: renamed from C1; footprint (none) -> Capacitor_SMD:CP_Elec_10x10.5
- ESP1: footprint MODULE_ESP32-DEVKITC-32D -> ESP32-DEVKITC-32D:MODULE_ESP32-DEVKITC-32D
- Q1: footprint (none) -> Package_TO_SOT_SMD:SOT-23_Handsoldering; symbol Device:Q_NPN_BCE -> Device:Q_NPN_BEC
- Q10, Q100, Q101, Q102, Q103, Q104, Q105, Q106, Q107, Q108, Q109, Q11, Q110, Q111, Q112, Q12, Q121, Q122, Q123, Q124, Q125, Q126, Q127, Q128, Q129, Q13, Q130, Q131, Q132, Q133, Q134, Q135, Q136, Q14, Q145, Q146, Q147, Q148, Q149, Q15, Q150, Q151, Q152, Q153, Q154, Q155, Q156, Q157, Q158, Q159, Q16, Q160, Q169, Q170, Q171, Q172, Q173, Q174, Q175, Q176, Q177, Q178, Q179, Q180, Q181, Q182, Q183, Q184, Q2, Q25, Q26, Q27, Q28, Q29, Q3, Q30, Q31, Q32, Q33, Q34, Q35, Q36, Q37, Q38, Q39, Q4, Q40, Q49, Q5, Q50, Q51, Q52, Q53, Q54, Q55, Q56, Q57, Q58, Q59, Q6, Q60, Q61, Q62, Q63, Q64, Q7, Q73, Q74, Q75, Q76, Q77, Q78, Q79, Q8, Q80, Q81, Q82, Q83, Q84, Q85, Q86, Q87, Q88, Q9, Q97, Q98, Q99: renamed from Q?; footprint (none) -> Package_TO_SOT_SMD:SOT-23_Handsoldering; symbol Device:Q_NPN_BCE -> Device:Q_NPN_BEC
- R1, R100, R101, R102, R103, R104, R145, R146, R147, R148, R149, R150, R151, R152, R193, R194, R195, R196, R197, R198, R199, R2, R200, R241, R242, R243, R244, R245, R246, R247, R248, R289, R290, R291, R292, R293, R294, R295, R296, R3, R337, R338, R339, R340, R341, R342, R343, R344, R4, R49, R5, R50, R51, R52, R53, R54, R55, R56, R6, R7, R8, R97, R98, R99: renamed from R?; footprint (none) -> Resistor_SMD:R_0805_2012Metric_Pad1.20x1.40mm_HandSolder
- R10, R105, R106, R107, R108, R109, R11, R110, R111, R112, R12, R13, R14, R15, R153, R154, R155, R156, R157, R158, R159, R16, R160, R201, R202, R203, R204, R205, R206, R207, R208, R249, R250, R251, R252, R253, R254, R255, R256, R297, R298, R299, R300, R301, R302, R303, R304, R345, R346, R347, R348, R349, R350, R351, R352, R57, R58, R59, R60, R61, R62, R63, R64, R9: renamed from R?; value 330 -> 665; footprint (none) -> Resistor_SMD:R_0805_2012Metric_Pad1.20x1.40mm_HandSolder
- R121, R122, R123, R124, R125, R126, R127, R128, R129, R130, R131, R132, R133, R134, R135, R136, R169, R170, R171, R172, R173, R174, R175, R176, R177, R178, R179, R180, R181, R182, R183, R184, R217, R218, R219, R220, R221, R222, R223, R224, R225, R226, R227, R228, R229, R230, R231, R232, R25, R26, R265, R266, R267, R268, R269, R27, R270, R271, R272, R273, R274, R275, R276, R277, R278, R279, R28, R280, R29, R30, R31, R313, R314, R315, R316, R317, R318, R319, R32, R320, R321, R322, R323, R324, R325, R326, R327, R328, R33, R34, R35, R36, R361, R362, R363, R364, R365, R366, R367, R368, R369, R37, R370, R371, R372, R373, R374, R375, R376, R38, R39, R40, R73, R74, R75, R76, R77, R78, R79, R80, R81, R82, R83, R84, R85, R86, R87, R88: renamed from R?; footprint (none) -> Resistor_SMD:R_0603_1608Metric_Pad0.98x0.95mm_HandSolder
- SW1, SW2, SW3, SW4, SW5: footprint (none) -> LED-Cube:SW_TACTILE_12x12mm
- TOUCH1, TOUCH2, TOUCH3, TOUCH4, TOUCH5: footprint (none) -> ESC_Pads:ESC_Pad_B
Connections:
- net labels added: +3V3, B1-1out, B1-2out, B1-3out, B1-4out, B1-5out, B1-6out, B1-7out, B1-8out, B2-1out, B2-2out, B2-3out, B2-4out, B2-5out, B2-6out, B2-7out, B2-8out, B3-1out, B3-2out, B3-3out, B3-4out, B3-5out, B3-6out, B3-7out, B3-8out, B4-1out, B4-2out, B4-3out, B4-4out, B4-5out, B4-6out, B4-7out, B4-8out, B5-1out, B5-2out, B5-3out, B5-4out, B5-5out, B5-6out, B5-7out, B5-8out, B6-1out, B6-2out, B6-3out, B6-4out, B6-5out, B6-6out, B6-7out, B6-8out, B7-1out, B7-2out, B7-3out, B7-4out, B7-5out, B7-6out, B7-7out, B7-8out, B8-1out, B8-2out, B8-3out, B8-4out, B8-5out, B8-6out, B8-7out, B8-8out, G1-1out, G1-2out, G1-3out, G1-4out, G1-5out, G1-6out, G1-7out, G1-8out, G2-1out, G2-2out, G2-3out, G2-4out, G2-5out, G2-6out, G2-7out, G2-8out, G3-1out, G3-2out, G3-3out, G3-4out, G3-5out, G3-6out, G3-7out, G3-8out, G4-1out, G4-2out, G4-3out, G4-4out, G4-5out, G4-6out, G4-7out, G4-8out, G5-1out, G5-2out, G5-3out, G5-4out, G5-5out, G5-6out, G5-7out, G5-8out, G6-1out, G6-2out, G6-3out, G6-4out, G6-5out, G6-6out, G6-7out, G6-8out, G7-1out, G7-2out, G7-3out, G7-4out, G7-5out, G7-6out, G7-7out, G7-8out, G8-1out, G8-2out, G8-3out, G8-4out, G8-5out, G8-6out, G8-7out, G8-8out, LED_strip, Layer1out, Layer2out, Layer3out, Layer4out, Layer5out, Layer6out, Layer7out, Layer8, Layer8out
- wire segments 846 -> 1289
- no-connect marks 0 -> 7
Other:
- moved on the sheet: C11, DC1, ESP1, R1, R10, R100, R101, R102, R103, R104, R105, R106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

Commit message: PCB update
Parts:
- C1, C10, C11, C12, C13, C14, C15, C16, C17, C18, C19, C2, C20, C21, C22, C23, C24, C25, C26, C27, C28, C29, C3, C30, C31, C32, C4, C5, C6, C7, C8, C9: renamed from C?; footprint (none) -> Capacitor_SMD:C_0603_1608Metric_Pad1.08x0.95mm_HandSolder
- R385, R386, R387, R388, R389, R390, R391, R392, R393, R394, R395, R396, R397, R398, R399, R400, R401, R402, R403, R404, R405, R406, R407, R408: renamed from R?; footprint (none) -> Resistor_SMD:R_0603_1608Metric_Pad0.98x0.95mm_HandSolder
- gave numbers to parts that had none: 48
- renumbered C1 to C33, C2 to C34, C3 to C35, C4 to C36, C5 to C37, C6 to C38, C7 to C39, C8 to C40, C9 to C41, C10 to C42, C11 to C43, C12 to C44, C13 to C45, C14 to C46, C15 to C47, C16 to C48, C17 to C49, C18 to C50, C19 to C51, C20 to C52, C21 to C53, C22 to C54, C23 to C55, C24 to C56, C25 to C57, C26 to C58, R385 to R409, R386 to R410, R387 to R411, R388 to R412, R389 to R413
Connections:
- wire segments 1289 -> 1337
- no-connect marks 7 -> 13
Other:
- moved on the sheet: C1, C17, C25, C33, C34, C35, C36, C37, C38, C39, C40, C41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

Commit message: PCB update
Parts:
- removed TOUCH1, TOUCH2, TOUCH3, TOUCH4, TOUCH5: ESC_Pad_B, ESC_Pads:ESC_Pad_B, symbol ESC_Pads:ESC_Pad_B
- added H1, H10, H100, H101, H102, H103, H104, H105, H106, H107, H108, H109, H11, H110, H111, H112, H113, H114, H115, H116, H117, H118, H119, H12, H120, H121, H122, H123, H124, H125, H126, H127, H128, H129, H13, H130, H131, H132, H133, H134, H135, H136, H137, H138, H139, H14, H140, H141, H142, H143, H144, H145, H146, H147, H148, H149, H15, H150, H151, H152, H153, H154, H155, H156, H157, H158, H159, H16, H160, H161, H162, H163, H164, H165, H166, H167, H168, H169, H17, H170, H171, H172, H173, H174, H175, H176, H177, H178, H179, H18, H180, H181, H182, H183, H184, H185, H186, H187, H188, H189, H19, H190, H191, H192, H193, H194, H195, H196, H197, H198, H199, H2, H20, H200, H21, H22, H23, H24, H25, H26, H27, H28, H29, H3, H30, H31, H32, H33, H34, H35, H36, H37, H38, H39, H4, H40, H41, H42, H43, H44, H45, H46, H47, H48, H49, H5, H50, H51, H52, H53, H54, H55, H56, H57, H58, H59, H6, H60, H61, H62, H63, H64, H65, H66, H67, H68, H69, H7, H70, H71, H72, H73, H74, H75, H76, H77, H78, H79, H8, H80, H81, H82, H83, H84, H85, H86, H87, H88, H89, H9, H90, H91, H92, H93, H94, H95, H96, H97, H98, H99: Wire_hole_1.2_2.5, LED-Cube:Wire_hole_1.5_2.8, symbol LED-Cube:Wire_hole_1.2_2.5
- added H201, H202, H203, H204: MountingHole, MountingHole:MountingHole_3.2mm_M3, symbol Mechanical:MountingHole
- added PAD1: DATA, LED-Cube:Solder_pad_3x3mm, symbol LED-Cube:Wire_pad
- added PAD10: 2BOUT, LED-Cube:Solder_pad_3x3mm, symbol LED-Cube:Wire_pad
- added PAD11: 2RIN, LED-Cube:Solder_pad_3x3mm, symbol LED-Cube:Wire_pad
- added PAD12: 2GIN, LED-Cube:Solder_pad_3x3mm, symbol LED-Cube:Wire_pad
- added PAD13: 2BIN, LED-Cube:Solder_pad_3x3mm, symbol LED-Cube:Wire_pad
- added PAD14: 3ROUT, LED-Cube:Solder_pad_3x3mm, symbol LED-Cube:Wire_pad
- added PAD15: 3GOUT, LED-Cube:Solder_pad_3x3mm, symbol LED-Cube:Wire_pad
- added PAD16: 3BOUT, LED-Cube:Solder_pad_3x3mm, symbol LED-Cube:Wire_pad
- added PAD17: 3RIN, LED-Cube:Solder_pad_3x3mm, symbol LED-Cube:Wire_pad
- added PAD18: 3GIN, LED-Cube:Solder_pad_3x3mm, symbol LED-Cube:Wire_pad
- added PAD19: 3BIN, LED-Cube:Solder_pad_3x3mm, symbol LED-Cube:Wire_pad
- added PAD2: 1ROUT, LED-Cube:Solder_pad_3x3mm, symbol LED-Cube:Wire_pad
- added PAD20: 4ROUT, LED-Cube:Solder_pad_3x3mm, symbol LED-Cube:Wire_pad
- added PAD21: 4GOUT, LED-Cube:Solder_pad_3x3mm, symbol LED-Cube:Wire_pad
- added PAD22: 4BOUT, LED-Cube:Solder_pad_3x3mm, symbol LED-Cube:Wire_pad
- added PAD23: 4RIN, LED-Cube:Solder_pad_3x3mm, symbol LED-Cube:Wire_pad
- added PAD24: 4GIN, LED-Cube:Solder_pad_3x3mm, symbol LED-Cube:Wire_pad
- added PAD25: 4BIN, LED-Cube:Solder_pad_3x3mm, symbol LED-Cube:Wire_pad
- added PAD26: 5ROUT, LED-Cube:Solder_pad_3x3mm, symbol LED-Cube:Wire_pad
- added PAD27: 5GOUT, LED-Cube:Solder_pad_3x3mm, symbol LED-Cube:Wire_pad
- added PAD28: 5BOUT, LED-Cube:Solder_pad_3x3mm, symbol LED-Cube:Wire_pad
- added PAD29: 5RIN, LED-Cube:Solder_pad_3x3mm, symbol LED-Cube:Wire_pad
- added PAD3: 1GOUT, LED-Cube:Solder_pad_3x3mm, symbol LED-Cube:Wire_pad
- added PAD30: 5GIN, LED-Cube:Solder_pad_3x3mm, symbol LED-Cube:Wire_pad
- added PAD31: 5BIN, LED-Cube:Solder_pad_3x3mm, symbol LED-Cube:Wire_pad
- added PAD32: 6ROUT, LED-Cube:Solder_pad_3x3mm, symbol LED-Cube:Wire_pad
- added PAD33: 6GOUT, LED-Cube:Solder_pad_3x3mm, symbol LED-Cube:Wire_pad
- added PAD34: 6BOUT, LED-Cube:Solder_pad_3x3mm, symbol LED-Cube:Wire_pad
- added PAD35: 6RIN, LED-Cube:Solder_pad_3x3mm, symbol LED-Cube:Wire_pad
- added PAD36: 6GIN, LED-Cube:Solder_pad_3x3mm, symbol LED-Cube:Wire_pad
- added PAD37: 6BIN, LED-Cube:Solder_pad_3x3mm, symbol LED-Cube:Wire_pad
- added PAD38: 7ROUT, LED-Cube:Solder_pad_3x3mm, symbol LED-Cube:Wire_pad
- added PAD39: 7GOUT, LED-Cube:Solder_pad_3x3mm, symbol LED-Cube:Wire_pad
- added PAD4: 1BOUT, LED-Cube:Solder_pad_3x3mm, symbol LED-Cube:Wire_pad
- added PAD40: 7BOUT, LED-Cube:Solder_pad_3x3mm, symbol LED-Cube:Wire_pad
- added PAD41: 7RIN, LED-Cube:Solder_pad_3x3mm, symbol LED-Cube:Wire_pad
- added PAD42: 7GIN, LED-Cube:Solder_pad_3x3mm, symbol LED-Cube:Wire_pad
- added PAD43: 7BIN, LED-Cube:Solder_pad_3x3mm, symbol LED-Cube:Wire_pad
- added PAD44: 8ROUT, LED-Cube:Solder_pad_3x3mm, symbol LED-Cube:Wire_pad
- added PAD45: 8GOUT, LED-Cube:Solder_pad_3x3mm, symbol LED-Cube:Wire_pad
- added PAD46: 8BOUT, LED-Cube:Solder_pad_3x3mm, symbol LED-Cube:Wire_pad
- added PAD47: LAYEROUT, LED-Cube:Solder_pad_3x3mm, symbol LED-Cube:Wire_pad
- added PAD48: 8RIN, LED-Cube:Solder_pad_3x3mm, symbol LED-Cube:Wire_pad
- added PAD49: 8GIN, LED-Cube:Solder_pad_3x3mm, symbol LED-Cube:Wire_pad
- added PAD5: 1RIN, LED-Cube:Solder_pad_3x3mm, symbol LED-Cube:Wire_pad
- added PAD50: 8BIN, LED-Cube:Solder_pad_3x3mm, symbol LED-Cube:Wire_pad
- added PAD51: LAYERIN, LED-Cube:Solder_pad_3x3mm, symbol LED-Cube:Wire_pad
- added PAD52, PAD53: Wire_pad, LED-Cube:Solder_pad_5x5mm, symbol LED-Cube:Wire_pad
- added PAD6: 1GIN, LED-Cube:Solder_pad_3x3mm, symbol LED-Cube:Wire_pad
- added PAD7: 1BIN, LED-Cube:Solder_pad_3x3mm, symbol LED-Cube:Wire_pad
- added PAD8: 2ROUT, LED-Cube:Solder_pad_3x3mm, symbol LED-Cube:Wire_pad
- added PAD9: 2GOUT, LED-Cube:Solder_pad_3x3mm, symbol LED-Cube:Wire_pad
- added PAD98, PAD99: Wire_pad, LED-Cube:Solder_pad_1.5x1.5mm, symbol LED-Cube:Wire_pad
- added R?: R_US, symbol Device:R_US
- added TOUCH1, TOUCH2, TOUCH3, TOUCH4, TOUCH5: Touch_pad, LED-Cube:Touch_pad, symbol LED-Cube:Touch_pad
- Q1, Q10, Q100, Q101, Q102, Q103, Q104, Q105, Q106, Q107, Q108, Q109, Q11, Q110, Q111, Q112, Q113, Q114, Q115, Q116, Q117, Q118, Q119, Q12, Q120, Q121, Q122, Q123, Q124, Q125, Q126, Q127, Q128, Q129, Q13, Q130, Q131, Q132, Q133, Q134, Q135, Q136, Q137, Q138, Q139, Q14, Q140, Q141, Q142, Q143, Q144, Q145, Q146, Q147, Q148, Q149, Q15, Q150, Q151, Q152, Q153, Q154, Q155, Q156, Q157, Q158, Q159, Q16, Q160, Q161, Q162, Q163, Q164, Q165, Q166, Q167, Q168, Q169, Q17, Q170, Q171, Q172, Q173, Q174, Q175, Q176, Q177, Q178, Q179, Q18, Q180, Q181, Q182, Q183, Q184, Q185, Q186, Q187, Q188, Q189, Q19, Q190, Q191, Q192, Q197, Q198, Q199, Q2, Q20, Q200, Q205, Q206, Q207, Q208, Q21, Q22, Q23, Q24, Q25, Q26, Q27, Q28, Q29, Q3, Q30, Q31, Q32, Q33, Q34, Q35, Q36, Q37, Q38, Q39, Q4, Q40, Q41, Q42, Q43, Q44, Q45, Q46, Q47, Q48, Q49, Q5, Q50, Q51, Q52, Q53, Q54, Q55, Q56, Q57, Q58, Q59, Q6, Q60, Q61, Q62, Q63, Q64, Q65, Q66, Q67, Q68, Q69, Q7, Q70, Q71, Q72, Q73, Q74, Q75, Q76, Q77, Q78, Q79, Q8, Q80, Q81, Q82, Q83, Q84, Q85, Q86, Q87, Q88, Q89, Q9, Q90, Q91, Q92, Q93, Q94, Q95, Q96, Q97, Q98, Q99: footprint Package_TO_SOT_SMD:SOT-23_Handsoldering -> Package_TO_SOT_SMD:SOT-23
Connections:
- net +5V: now also C1.1, C10.1, C11.1, C12.1, C13.1, C14.1, C15.1, C16.1, C17.1, C18.1, C19.1, C2.1, C20.1, C21.1, C22.1, C23.1, C24.1, C25.1, C26.1, C27.1, C28.1, C29.1, C3.1, C30.1, C31.1, C32.1, C4.1, C5.1, C6.1, C7.1, C8.1, C9.1, D1.1 (VDD), D10.1 (VDD), D11.1 (VDD), D12.1 (VDD), D13.1 (VDD), D14.1 (VDD), D15.1 (VDD), D16.1 (VDD)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
- net GND: now also C1.2, C10.2, C11.2, C12.2, C13.2, C14.2, C15.2, C16.2, C17.2, C18.2, C19.2, C2.2, C20.2, C21.2, C22.2, C23.2, C24.2, C25.2, C26.2, C27.2, C28.2, C29.2, C3.2, C30.2, C31.2, C32.2, C4.2, C5.2, C6.2, C7.2, C8.2, C9.2, D1.3 (VSS), D10.3 (VSS), D11.3 (VSS), D12.3 (VSS), D13.3 (VSS), D14.3 (VSS), D15.3 (VSS), D16.3 (VSS)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
- net LED_strip: now also R?.2
- net Layer7: no longer U1.7 (QH)
- net Layer8: now also U1.7 (QH)
- net Touch1: now also SW1.2, TOUCH1.1
- net Touch2: now also SW2.2, TOUCH2.1
- net Touch3: now also SW3.2, TOUCH3.1
- net Touch4: now also SW4.2, TOUCH4.1
- net Touch5: now also SW5.2, TOUCH5.1
- net at U1.9 (QH'): now also PAD47.1; no longer U2.14 (SER)
- net at U2.9 (QH'): now also PAD2.1; no longer U3.14 (SER)
- net at U3.9 (QH'): now also PAD3.1; no longer U4.14 (SER)
- net at U4.9 (QH'): now also PAD4.1; no longer U5.14 (SER)
- net at U5.9 (QH'): now also PAD8.1; no longer U6.14 (SER)
- net at U6.9 (QH'): now also PAD9.1; no longer U7.14 (SER)
- net at U7.9 (QH'): now also PAD10.1; no longer U8.14 (SER)
- net at U8.9 (QH'): now also PAD14.1; no longer U9.14 (SER)
- net at U9.9 (QH'): now also PAD15.1; no longer U10.14 (SER)
- net at U10.9 (QH'): now also PAD16.1; no longer U11.14 (SER)
- net at U11.9 (QH'): now also PAD20.1; no longer U12.14 (SER)
- net at U12.9 (QH'): now also PAD21.1; no longer U13.14 (SER)
- net at U13.9 (QH'): now also PAD22.1; no longer U14.14 (SER)
- net at U14.9 (QH'): now also PAD26.1; no longer U15.14 (SER)
- net at U15.9 (QH'): now also PAD27.1; no longer U16.14 (SER)
- net at U16.9 (QH'): now also PAD28.1; no longer U17.14 (SER)
- net at U17.9 (QH'): now also PAD32.1; no longer U18.14 (SER)
- net at U18.9 (QH'): now also PAD33.1; no longer U19.14 (SER)
- net at U19.9 (QH'): now also PAD34.1; no longer U20.14 (SER)
- net at U20.9 (QH'): now also PAD38.1; no longer U21.14 (SER)
- net at U21.9 (QH'): now also PAD39.1; no longer U22.14 (SER)
- net at U22.9 (QH'): now also PAD40.1; no longer U23.14 (SER)
- net at U23.9 (QH'): now also PAD44.1; no longer U24.14 (SER)
- net at U24.9 (QH'): now also PAD45.1; no longer U25.14 (SER)
- net at U25.9 (QH'): now also PAD46.1
- net at D28.2 (DOUT): now also PAD98.1; no longer D29.4 (DIN)
- net B1-1out: no longer names the net of R17.1
- net B1-1out: now also H17.~
- net B1-2out: no longer names the net of R18.1
- net B1-2out: now also H18.~
- net B1-3out: no longer names the net of R19.1
- net B1-3out: now also H19.~
- net B1-4out: no longer names the net of R20.1
- net B1-4out: now also H20.~
- net B1-5out: no longer names the net of R21.1
- net B1-5out: now also H21.~
- net B1-6out: no longer names the net of R22.1
- net B1-6out: now also H22.~
- net B1-7out: no longer names the net of R23.1
- net B1-7out: now also H23.~
- net B1-8out: no longer names the net of R24.1
- net B1-8out: now also H24.~
- net B2-1out: no longer names the net of R65.1
- net B2-1out: now also H41.~
- net B2-2out: no longer names the net of R66.1
- net B2-2out: now also H42.~
- net B2-3out: no longer names the net of R67.1
- net B2-3out: now also H43.~
- net B2-4out: no longer names the net of R68.1
- net B2-4out: now also H44.~
- net B2-5out: no longer names the net of R69.1
- net B2-5out: now also H45.~
- net B2-6out: no longer names the net of R70.1
- net B2-6out: now also H46.~
- net B2-7out: no longer names the net of R71.1
- net B2-7out: now also H47.~
- net B2-8out: no longer names the net of R72.1
- net B2-8out: now also H48.~
- net B3-1out: no longer names the net of R113.1
- net B3-1out: now also H65.~
- net B3-2out: no longer names the net of R114.1
- net B3-2out: now also H66.~
- net B3-3out: no longer names the net of R115.1
- net B3-3out: now also H67.~
- net B3-4out: no longer names the net of R116.1
- net B3-4out: now also H68.~
- net B3-5out: no longer names the net of R117.1
- net B3-5out: now also H69.~
- net B3-6out: no longer names the net of R118.1
- net B3-6out: now also H70.~
- net B3-7out: no longer names the net of R119.1
- net B3-7out: now also H71.~
- net B3-8out: no longer names the net of R120.1
- net B3-8out: now also H72.~
- net B4-1out: no longer names the net of R161.1
- net B4-1out: now also H89.~
- net B4-2out: no longer names the net of R162.1
- net B4-2out: now also H90.~
- net B4-3out: no longer names the net of R163.1
- net B4-3out: now also H91.~
- net B4-4out: no longer names the net of R164.1
- net B4-4out: now also H92.~
- net B4-5out: no longer names the net of R165.1
- net B4-5out: now also H93.~
- net B4-6out: no longer names the net of R166.1
- net B4-6out: now also H94.~
- net B4-7out: no longer names the net of R167.1
- net B4-7out: now also H95.~
- net B4-8out: no longer names the net of R168.1
- net B4-8out: now also H96.~
- net B5-1out: no longer names the net of R209.1
- net B5-1out: now also H113.~
- net B5-2out: no longer names the net of R210.1
- net B5-2out: now also H114.~
- net B5-3out: no longer names the net of R211.1
- net B5-3out: now also H115.~
- net B5-4out: no longer names the net of R212.1
- net B5-4out: now also H116.~
- net B5-5out: no longer names the net of R213.1
- net B5-5out: now also H117.~
- net B5-6out: no longer names the net of R214.1
- net B5-6out: now also H118.~
- net B5-7out: no longer names the net of R215.1
- net B5-7out: now also H119.~
- net B5-8out: no longer names the net of R216.1
- net B5-8out: now also H120.~
- net B6-1out: no longer names the net of R257.1
- net B6-1out: now also H137.~
- net B6-2out: no longer names the net of R258.1
- net B6-2out: now also H138.~
- net B6-3out: no longer names the net of R259.1
- net B6-3out: now also H139.~
- net B6-4out: no longer names the net of R260.1
- net B6-4out: now also H140.~
- net B6-5out: no longer names the net of R261.1
- net B6-5out: now also H141.~
- net B6-6out: no longer names the net of R262.1
- net B6-6out: now also H142.~
- net B6-7out: no longer names the net of R263.1
- net B6-7out: now also H143.~
- net B6-8out: no longer names the net of R264.1
- net B6-8out: now also H144.~
- net B7-1out: no longer names the net of R305.1
- net B7-1out: now also H161.~
- net B7-2out: no longer names the net of R306.1
- net B7-2out: now also H162.~
- net B7-3out: no longer names the net of R307.1
- net B7-3out: now also H163.~
- net B7-4out: no longer names the net of R308.1
- net B7-4out: now also H164.~
- net B7-5out: no longer names the net of R309.1
- net B7-5out: now also H165.~
- net B7-6out: no longer names the net of R310.1
- net B7-6out: now also H166.~
- net B7-7out: no longer names the net of R311.1
- net B7-7out: now also H167.~
- net B7-8out: no longer names the net of R312.1
- net B7-8out: now also H168.~
- net B8-1out: no longer names the net of R353.1
- net B8-1out: now also H185.~
- net B8-2out: no longer names the net of R354.1
- net B8-2out: now also H186.~
- net B8-3out: no longer names the net of R355.1
- net B8-3out: now also H187.~
- net B8-4out: no longer names the net of R356.1
- net B8-4out: now also H188.~
- net B8-5out: no longer names the net of R357.1
- net B8-5out: now also H189.~
- net B8-6out: no longer names the net of R358.1
- net B8-6out: now also H190.~
- net B8-7out: no longer names the net of R359.1
- net B8-7out: now also H191.~
- net B8-8out: no longer names the net of R360.1
- net B8-8out: now also H192.~
- net G1-1out: no longer names the net of R9.1
- net G1-1out: now also H9.~
- net G1-2out: no longer names the net of R10.1
- net G1-2out: now also H10.~
- net G1-3out: no longer names the net of R11.1
- net G1-3out: now also H11.~
- net G1-4out: no longer names the net of R12.1
- net G1-4out: now also H12.~
- net G1-5out: no longer names the net of R13.1
- net G1-5out: now also H13.~
- net G1-6out: no longer names the net of R14.1
- net G1-6out: now also H14.~
- net G1-7out: no longer names the net of R15.1
- net G1-7out: now also H15.~
- net G1-8out: no longer names the net of R16.1
- net G1-8out: now also H16.~
- net G2-1out: no longer names the net of R57.1
- net G2-1out: now also H33.~
- net G2-2out: no longer names the net of R58.1
- net G2-2out: now also H34.~
- net G2-3out: no longer names the net of R59.1
- net G2-3out: now also H35.~
- net G2-4out: no longer names the net of R60.1
- net G2-4out: now also H36.~
- net G2-5out: no longer names the net of R61.1
- net G2-5out: now also H37.~
- net G2-6out: no longer names the net of R62.1
- net G2-6out: now also H38.~
- net G2-7out: no longer names the net of R63.1
- net G2-7out: now also H39.~
- net G2-8out: no longer names the net of R64.1
- net G2-8out: now also H40.~
- net G3-1out: no longer names the net of R105.1
- net G3-1out: now also H57.~
- net G3-2out: no longer names the net of R106.1
- net G3-2out: now also H58.~
- net G3-3out: no longer names the net of R107.1
- net G3-3out: now also H59.~
- net G3-4out: no longer names the net of R108.1
- net G3-4out: now also H60.~
- net G3-5out: no longer names the net of R109.1
- net G3-5out: now also H61.~
- net G3-6out: no longer names the net of R110.1
- net G3-6out: now also H62.~
- net G3-7out: no longer names the net of R111.1
- net G3-7out: now also H63.~
- net G3-8out: no longer names the net of R112.1
- net G3-8out: now also H64.~
- net G4-1out: no longer names the net of R153.1
- net G4-1out: now also H81.~
- net G4-2out: no longer names the net of R154.1
- net G4-2out: now also H82.~
- net G4-3out: no longer names the net of R155.1
- net G4-3out: now also H83.~
- net G4-4out: no longer names the net of R156.1
- net G4-4out: now also H84.~
- net G4-5out: no longer names the net of R157.1
- net G4-5out: now also H85.~
- net G4-6out: no longer names the net of R158.1
- net G4-6out: now also H86.~
- net G4-7out: no longer names the net of R159.1
- net G4-7out: now also H87.~
- net G4-8out: no longer names the net of R160.1
- net G4-8out: now also H88.~
- net G5-1out: no longer names the net of R201.1
- net G5-1out: now also H105.~
- net G5-2out: no longer names the net of R202.1
- net G5-2out: now also H106.~
- net G5-3out: no longer names the net of R203.1
- net G5-3out: now also H107.~
- net G5-4out: no longer names the net of R204.1
- net G5-4out: now also H108.~
- net G5-5out: no longer names the net of R205.1
- net G5-5out: now also H109.~
- net G5-6out: no longer names the net of R206.1
- net G5-6out: now also H110.~
- net G5-7out: no longer names the net of R207.1
- net G5-7out: now also H111.~
- net G5-8out: no longer names the net of R208.1
- net G5-8out: now also H112.~
- net G6-1out: no longer names the net of R249.1
- net G6-1out: now also H129.~
- net G6-2out: no longer names the net of R250.1
- net G6-2out: now also H130.~
- net G6-3out: no longer names the net of R251.1
- net G6-3out: now also H131.~
- net G6-4out: no longer names the net of R252.1
- net G6-4out: now also H132.~
- net G6-5out: no longer names the net of R253.1
- net G6-5out: now also H133.~
- net G6-6out: no longer names the net of R254.1
- net G6-6out: now also H134.~
- net G6-7out: no longer names the net of R255.1
- net G6-7out: now also H135.~
- net G6-8out: no longer names the net of R256.1
- net G6-8out: now also H136.~
- net G7-1out: no longer names the net of R297.1
- net G7-1out: now also H153.~
- net G7-2out: no longer names the net of R298.1
- net G7-2out: now also H154.~
- net G7-3out: no longer names the net of R299.1
- net G7-3out: now also H155.~
- net G7-4out: no longer names the net of R300.1
- net G7-4out: now also H156.~
- net G7-5out: no longer names the net of R301.1
- net G7-5out: now also H157.~
- net G7-6out: no longer names the net of R302.1
- net G7-6out: now also H158.~
- net G7-7out: no longer names the net of R303.1
- net G7-7out: now also H159.~
- net G7-8out: no longer names the net of R304.1
- net G7-8out: now also H160.~
- net G8-1out: no longer names the net of R345.1
- net G8-1out: now also H177.~
- net G8-2out: no longer names the net of R346.1
- net G8-2out: now also H178.~
- net G8-3out: no longer names the net of R347.1
- net G8-3out: now also H179.~
- net G8-4out: no longer names the net of R348.1
- net G8-4out: now also H180.~
- net G8-5out: no longer names the net of R349.1
- net G8-5out: now also H181.~
- net G8-6out: no longer names the net of R350.1
- net G8-6out: now also H182.~
- net G8-7out: no longer names the net of R351.1
- net G8-7out: now also H183.~
- net G8-8out: no longer names the net of R352.1
- net G8-8out: now also H184.~
- net Layer1out: no longer names the net of Q193.2 (S)
- net Layer1out: now also H193.~
- net Layer2out: no longer names the net of Q194.2 (S)
- net Layer2out: now also H194.~
- net Layer3out: no longer names the net of Q195.2 (S)
- net Layer3out: now also H195.~
- net Layer4out: no longer names the net of Q196.2 (S)
- net Layer4out: now also H196.~
- net Layer5out: no longer names the net of Q201.2 (S)
- net Layer5out: now also H197.~
- net Layer6out: no longer names the net of Q202.2 (S)
- net Layer6out: now also H198.~
- net Layer7out: no longer names the net of Q203.2 (S)
- net Layer7out: now also H199.~
- net Layer8out: no longer names the net of Q204.2 (S)
- net Layer8out: now also H200.~
- net R1-1out: no longer names the net of R1.1
- net R1-1out: now also H1.~
- net R1-2out: no longer names the net of R2.1
- net R1-2out: now also H2.~
- net R1-3out: no longer names the net of R3.1
- net R1-3out: now also H3.~
- net R1-4out: no longer names the net of R4.1
- net R1-4out: now also H4.~
- net R1-5out: no longer names the net of R5.1
- net R1-5out: now also H5.~
- net R1-6out: no longer names the net of R6.1
- net R1-6out: now also H6.~
- net R1-7out: no longer names the net of R7.1
- net R1-7out: now also H7.~
- net R1-8out: no longer names the net of R8.1
- net R1-8out: now also H8.~
- net R2-1out: no longer names the net of R49.1
- net R2-1out: now also H25.~
- net R2-2out: no longer names the net of R50.1
- net R2-2out: now also H26.~
- net R2-3out: no longer names the net of R51.1
- net R2-3out: now also H27.~
- net R2-4out: no longer names the net of R52.1
- net R2-4out: now also H28.~
- net R2-5out: no longer names the net of R53.1
- net R2-5out: now also H29.~
- net R2-6out: no longer names the net of R54.1
- net R2-6out: now also H30.~
- net R2-7out: no longer names the net of R55.1
- net R2-7out: now also H31.~
- net R2-8out: no longer names the net of R56.1
- net R2-8out: now also H32.~
- net R3-1out: no longer names the net of R97.1
- net R3-1out: now also H49.~
- net R3-2out: no longer names the net of R98.1
- net R3-2out: now also H50.~
- net R3-3out: no longer names the net of R99.1
- net R3-3out: now also H51.~
- net R3-4out: no longer names the net of R100.1
- net R3-4out: now also H52.~
- net R3-5out: no longer names the net of R101.1
- net R3-5out: now also H53.~
- net R3-6out: no longer names the net of R102.1
- net R3-6out: now also H54.~
- net R3-7out: no longer names the net of R103.1
- net R3-7out: now also H55.~
- net R3-8out: no longer names the net of R104.1
- net R3-8out: now also H56.~
- net R4-1out: no longer names the net of R145.1
- net R4-1out: now also H73.~
- net R4-2out: no longer names the net of R146.1
- net R4-2out: now also H74.~
- net R4-3out: no longer names the net of R147.1
- net R4-3out: now also H75.~
- net R4-4out: no longer names the net of R148.1
- net R4-4out: now also H76.~
- net R4-5out: no longer names the net of R149.1
- net R4-5out: now also H77.~
- net R4-6out: no longer names the net of R150.1
- net R4-6out: now also H78.~
- net R4-7out: no longer names the net of R151.1
- net R4-7out: now also H79.~
- net R4-8out: no longer names the net of R152.1
- net R4-8out: now also H80.~
- net R5-1out: no longer names the net of R193.1
- net R5-1out: now also H97.~
- net R5-2out: no longer names the net of R194.1
- net R5-2out: now also H98.~
- net R5-3out: no longer names the net of R195.1
- net R5-3out: now also H99.~
- net R5-4out: no longer names the net of R196.1
- net R5-4out: now also H100.~
- net R5-5out: no longer names the net of R197.1
- net R5-5out: now also H101.~
- net R5-6out: no longer names the net of R198.1
- net R5-6out: now also H102.~
- net R5-7out: no longer names the net of R199.1
- net R5-7out: now also H103.~
- net R5-8out: no longer names the net of R200.1
- net R5-8out: now also H104.~
- net R6-1out: no longer names the net of R241.1
- net R6-1out: now also H121.~
- net R6-2out: no longer names the net of R242.1
- net R6-2out: now also H122.~
- net R6-3out: no longer names the net of R243.1
- net R6-3out: now also H123.~
- net R6-4out: no longer names the net of R244.1
- net R6-4out: now also H124.~
- net R6-5out: no longer names the net of R245.1
- net R6-5out: now also H125.~
- net R6-6out: no longer names the net of R246.1
- net R6-6out: now also H126.~
- net R6-7out: no longer names the net of R247.1
- net R6-7out: now also H127.~
- net R6-8out: no longer names the net of R248.1
- net R6-8out: now also H128.~
- net R7-1out: no longer names the net of R289.1
- net R7-1out: now also H145.~
- net R7-2out: no longer names the net of R290.1
- net R7-2out: now also H146.~
- net R7-3out: no longer names the net of R291.1
- net R7-3out: now also H147.~
- net R7-4out: no longer names the net of R292.1
- net R7-4out: now also H148.~
- net R7-5out: no longer names the net of R293.1
- net R7-5out: now also H149.~
- net R7-6out: no longer names the net of R294.1
- net R7-6out: now also H150.~
- net R7-7out: no longer names the net of R295.1
- net R7-7out: now also H151.~
- net R7-8out: no longer names the net of R296.1
- net R7-8out: now also H152.~
- net R8-1out: no longer names the net of R337.1
- net R8-1out: now also H169.~
- net R8-2out: no longer names the net of R338.1
- net R8-2out: now also H170.~
- net R8-3out: no longer names the net of R339.1
- net R8-3out: now also H171.~
- net R8-4out: no longer names the net of R340.1
- net R8-4out: now also H172.~
- net R8-5out: no longer names the net of R341.1
- net R8-5out: now also H173.~
- net R8-6out: no longer names the net of R342.1
- net R8-6out: now also H174.~
- net R8-7out: no longer names the net of R343.1
- net R8-7out: now also H175.~
- net R8-8out: no longer names the net of R344.1
- net R8-8out: now also H176.~
- net serial_data_in: no longer names the net of ESP1.21 (IO23), R409.1
- net serial_data_in: now also PAD1.1; no longer U1.14 (SER)
- new net: PAD51.1, U1.14 (SER)
- new net: PAD5.1, U2.14 (SER)
- new net: PAD6.1, U3.14 (SER)
- new net: PAD7.1, U4.14 (SER)
- new net: PAD11.1, U5.14 (SER)
- new net: PAD12.1, U6.14 (SER)
- new net: PAD13.1, U7.14 (SER)
- new net: PAD17.1, U8.14 (SER)
- new net: PAD18.1, U9.14 (SER)
- new net: PAD19.1, U10.14 (SER)
- new net: PAD23.1, U11.14 (SER)
- new net: PAD24.1, U12.14 (SER)
- new net: PAD25.1, U13.14 (SER)
- new net: PAD29.1, U14.14 (SER)
- new net: PAD30.1, U15.14 (SER)
- new net: PAD31.1, U16.14 (SER)
- new net: PAD35.1, U17.14 (SER)
- new net: PAD36.1, U18.14 (SER)
- new net: PAD37.1, U19.14 (SER)
- new net: PAD41.1, U20.14 (SER)
- new net: PAD42.1, U21.14 (SER)
- new net: PAD43.1, U22.14 (SER)
- new net: PAD48.1, U23.14 (SER)
- new net: PAD49.1, U24.14 (SER)
- new net: PAD50.1, U25.14 (SER)
- new net: D29.4 (DIN), PAD99.1
- no-connect marks 13 -> 23
Other:
- moved on the sheet: C33, U1

Commit message: Alost finished PCB update
Parts:
- added PAD54, PAD55: Wire_pad, LED-Cube:Solder_pad_1.5x1.5mm, symbol LED-Cube:Wire_pad
- added TB1: Terminal_block, LED-Cube:Terminal_block, symbol LED-Cube:Terminal_block
- R414: renamed from R?; value R_US -> 10k; footprint (none) -> Resistor_SMD:R_0603_1608Metric_Pad0.98x0.95mm_HandSolder
Connections:
- net +5V: now also TB1.1
- net GND: now also TB1.2
- net LED_strip: now also PAD54.1; no longer D1.4 (DIN)
- new net: D1.4 (DIN), PAD55.1
Other:
- moved on the sheet: DC1
Changed lines of the file:
@@
 L Connector:Barrel_Jack_Switch DC1
 U 1 1 618C7052
-P 1650 7500
-F 0 "DC1" H 1707 7817 50  0000 C CNN
-F 1 "Barrel_Jack_Switch" H 1707 7726 50  0000 C CNN
-F 2 "Connector_BarrelJack:BarrelJack_Horizontal" H 1700 7460 50  0001 C CNN
-F 3 "~" H 1700 7460 50  0001 C CNN
-	1    1650 7500
+P 1500 7250
+F 0 "DC1" H 1557 7567 50  0000 C CNN
+F 1 "Barrel_Jack_Switch" H 1557 7476 50  0000 C CNN
+F 2 "Connector_BarrelJack:BarrelJack_Horizontal" H 1550 7210 50  0001 C CNN
+F 3 "~" H 1550 7210 50  0001 C CNN
+	1    1500 7250
 	1    0    0    -1
 $EndComp
@@
 L power:GND #PWR0256
 U 1 1 618C333D
-P 1950 7600
-F 0 "#PWR0256" H 1950 7350 50  0001 C CNN
-F 1 "GND" V 1955 7472 50  0000 R CNN
-F 2 "" H 1950 7600 50  0001 C CNN
-F 3 "" H 1950 7600 50  0001 C CNN
-	1    1950 7600
+P 1800 7350
+F 0 "#PWR0256" H 1800 7100 50  0001 C CNN
+F 1 "GND" V 1805 7222 50  0000 R CNN
+F 2 "" H 1800 7350 50  0001 C CNN
+F 3 "" H 1800 7350 50  0001 C CNN
+	1    1800 7350
 	0    -1   -1   0
 $EndComp
@@
 L power:+5V #PWR0253
 U 1 1 618C1D3E
-P 1950 7400
-F 0 "#PWR0253" H 1950 7250 50  0001 C CNN
-F 1 "+5V" V 1965 7528 50  0000 L CNN
-F 2 "" H 1950 7400 50  0001 C CNN
-F 3 "" H 1950 7400 50  0001 C CNN
-	1    1950 7400
+P 1800 7150
+F 0 "#PWR0253" H 1800 7000 50  0001 C CNN
+F 1 "+5V" V 1815 7278 50  0000 L CNN
+F 2 "" H 1800 7150 50  0001 C CNN
+F 3 "" H 1800 7150 50  0001 C CNN
+	1    1800 7150
 	0    1    1    0
 $EndComp
@@
 	1    0    0    -1
 $EndComp
-Text GLabel 11850 6400 0    50   Input ~ 0
+Text GLabel 11350 6400 0    50   Input ~ 0
 LED_strip
 $Comp
@@
 $EndComp
 Wire Wire Line
-	1950 7500 1950 7600
-Connection ~ 1950 7600
+	1800 7250 1800 7350
+Connection ~ 1800 7350
 Connection ~ 14800 9100
 Connection ~ 14800 8500
@@
 Wire Wire Line
 	1400 6000 1150 6000
+$Comp
+L Device:R_US R414
+U 1 1 6FD02D22
+P 1150 5850
+F 0 "R414" H 1218 5896 50  0000 L CNN
+F 1 "10k" H 1218 5805 50  0000 L CNN
+F 2 "Resistor_SMD:R_0603_1608Metric_Pad0.98x0.95mm_HandSolder" V 1190 5840 50  0001 C CNN
+F 3 "~" H 1150 5850 50  0001 C CNN
+	1    1150 5850
+	1    0    0    -1
+$EndComp
+Connection ~ 1150 6000
+Wire Wire Line
+	1150 6000 1050 6000
+$Comp
+L power:GND #PWR0317
+U 1 1 6FD0902B
+P 1150 5700
+F 0 "#PWR0317" H 1150 5450 50  0001 C CNN
+F 1 "GND" H 1155 5527 50  0000 C CNN
+F 2 "" H 1150 5700 50  0001 C CNN
+F 3 "" H 1150 5700 50  0001 C CNN
+	1    1150 5700
+	-1   0    0    1
+$EndComp
+$Comp
+L LED-Cube:Terminal_block TB1
+U 1 1 61EB8D37
+P 1550 7650
+F 0 "TB1" V 1550 8050 50  0000 R CNN
+F 1 "Terminal_block" V 1650 8450 50  0000 R CNN
+F 2 "LED-Cube:Terminal_block" H 1550 7650 50  0001 C CNN
+F 3 "" H 1550 7650 50  0001 C CNN
+	1    1550 7650
+	0    -1   -1   0
+$EndComp
+$Comp
+L power:+5V #PWR0318
+U 1 1 626C15A3
+P 1650 7550
+F 0 "#PWR0318" H 1650 7400 50  0001 C CNN
+F 1 "+5V" V 1665 7678 50  0000 L CNN
+F 2 "" H 1650 7550 50  0001 C CNN
+F 3 "" H 1650 7550 50  0001 C CNN
+	1    1650 7550
+	0    1    1    0
+$EndComp
+$Comp
+L power:GND #PWR0319
+U 1 1 626C7999
+P 1650 7750
+F 0 "#PWR0319" H 1650 7500 50  0001 C CNN
+F 1 "GND" V 1655 7622 50  0000 R CNN
+F 2 "" H 1650 7750 50  0001 C CNN
+F 3 "" H 1650 7750 50  0001 C CNN
+	1    1650 7750
+	0    -1   -1   0
+$EndComp
+$Comp
+L LED-Cube:Wire_pad PAD54
+U 1 1 62CB0BEC
+P 11400 6450
+F 0 "PAD54" V 11650 6350 50  0000 L CNN
+F 1 "Wire_pad" V 11550 6250 50  0000 L CNN
+F 2 "LED-Cube:Solder_pad_1.5x1.5mm" H 11400 6450 50  0001 C CNN
+F 3 "" H 11400 6450 50  0001 C CNN
+	1    11400 6450
+	0    1    1    0
+$EndComp
+$Comp
+L LED-Cube:Wire_pad PAD55
+U 1 1 62CB84D9
+P 11800 6450
+F 0 "PAD55" V 12050 6350 50  0000 L CNN
+F 1 "Wire_pad" V 11950 6250 50  0000 L CNN
+F 2 "LED-Cube:Solder_pad_1.5x1.5mm" H 11800 6450 50  0001 C CNN
+F 3 "" H 11800 6450 50  0001 C CNN
+	1    11800 6450
+	0    1    1    0
+$EndComp
+Wire Wire Line
+	11350 6400 11400 6400
+Wire Wire Line
+	11400 6400 11400 6450
+Wire Wire Line
+	11850 6400 11800 6400
+Wire Wire Line
+	11800 6400 11800 6450
 Wire Bus Line
 	11300 3500 16750 3500
@@
 Wire Bus Line
 	20850 3750 24450 3750
-$Comp
-L Device:R_US R?
-U 1 1 6FD02D22
-P 1150 5850
-F 0 "R?" H 1218 5896 50  0000 L CNN
-F 1 "R_US" H 1218 5805 50  0000 L CNN
-F 2 "" V 1190 5840 50  0001 C CNN
-F 3 "~" H 1150 5850 50  0001 C CNN
-	1    1150 5850
-	1    0    0    -1
-$EndComp
-Connection ~ 1150 6000
-Wire Wire Line
-	1150 6000 1050 6000
-$Comp
-L power:GND #PWR?
-U 1 1 6FD0902B
-P 1150 5700
-F 0 "#PWR?" H 1150 5450 50  0001 C CNN
-F 1 "GND" H 1155 5527 50  0000 C CNN
-F 2 "" H 1150 5700 50  0001 C CNN
-F 3 "" H 1150 5700 50  0001 C CNN
-	1    1150 5700
-	-1   0    0    1
-$EndComp
 $EndSCHEMATC

Commit message: FINAL PCB update and some middle testing code update
Parts:
- added C59, C60: 0.1u, Capacitor_SMD:C_0603_1608Metric_Pad1.08x0.95mm_HandSolder, symbol Device:C
- added U26: TXB0108PWR, Package_SO:TSSOP-20_4.4x6.5mm_P0.65mm, symbol LED-Cube:TXB0108PWR
- R1, R100, R101, R102, R103, R104, R145, R146, R147, R148, R149, R150, R151, R152, R193, R194, R195, R196, R197, R198, R199, R2, R200, R241, R242, R243, R244, R245, R246, R247, R248, R289, R290, R291, R292, R293, R294, R295, R296, R3, R337, R338, R339, R340, R341, R342, R343, R344, R4, R49, R5, R50, R51, R52, R53, R54, R55, R56, R6, R7, R8, R97, R98, R99: value 330 -> 220
Connections:
- net +3V3: now also C59.2, U26.10 (OE), U26.2 (VCCA)
- net +5V: now also C60.2, U26.19 (VCCB)
- net GND: now also C59.1, C60.1, U26.11 (GND), U26.8 (A7), U26.9 (A8)
- net LED_strip: now also U26.14 (B6); no longer ESP1.12 (IO14), R414.2
- net output_enable: now also U26.16 (B4); no longer ESP1.31 (IO16), R410.2
- net reset: now also U26.15 (B5); no longer ESP1.32 (IO4), R413.1
- net shifting_clock: now also U26.18 (B2); no longer ESP1.28 (IO18), R412.2
- net update_latch: now also U26.17 (B3); no longer ESP1.30 (IO17), R411.2
- net at ESP1.21 (IO23), R409.1: now also U26.1 (A1); no longer PAD1.1
- new net: ESP1.12 (IO14), R414.2, U26.7 (A6)
- new net: ESP1.28 (IO18), R412.2, U26.3 (A2)
- new net: ESP1.30 (IO17), R411.2, U26.4 (A3)
- new net: ESP1.31 (IO16), R410.2, U26.5 (A4)
- new net: ESP1.32 (IO4), R413.1, U26.6 (A5)
- new net: PAD1.1, U26.20 (B1)
- no-connect marks 23 -> 25
Other:
- moved on the sheet: C1, C17, C25, C33, C34, C35, C36, C37, C38, C39, C40, C41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
